File: hardware/led_stairs_controller.kicad_sch (KiCad schematic)
At the start: 59 parts, among them J1 Conn_02x10_Odd_Even, J10 Screw_Terminal_01x06, J11 Screw_Terminal_01x06, J12 Screw_Terminal_01x06, J13 Screw_Terminal_01x06, J14 Screw_Terminal_01x06, J15 Screw_Terminal_01x06, J16 Screw_Terminal_01x06, J17 Screw_Terminal_01x06, J18 Screw_Terminal_01x06, J19 Screw_Terminal_01x06, J2 Screw_Terminal_01x06, J3 Screw_Terminal_01x06, J4 Screw_Terminal_01x06, J5 Screw_Terminal_01x06, J6 Screw_Terminal_01x06, J7 Screw_Terminal_01x06, J8 Screw_Terminal_01x06, J9 Screw_Terminal_01x06, Q1 QM6006D, Q10 QM6006D, Q11 QM6006D, Q12 QM6006D, Q13 QM6006D, Q14 QM6006D, Q15 QM6006D, Q16 QM6006D, Q2 QM6006D, Q3 QM6006D, Q4 QM6006D, Q5 QM6006D, Q6 QM6006D, Q7 QM6006D, Q8 QM6006D, Q9 QM6006D, U1 PCA9635

Commit message: update
Parts:
- J3: footprint TerminalBlock_TE-Connectivity:TerminalBlock_TE_282834-6_1x06_P2.54mm_Horizontal -> TerminalBlock_Phoenix:TerminalBlock_Phoenix_MKDS-1,5-6_1x06_P5.00mm_Horizontal

Commit message: update
update
Parts:
- removed J10, J11, J12, J13, J14, J15, J16, J17, J18, J19, J2, J4, J5, J6, J7, J8, J9: Screw_Terminal_01x06, TerminalBlock_TE-Connectivity:TerminalBlock_TE_282834-6_1x06_P2.54mm_Horizontal, symbol Connector:Screw_Terminal_01x06
- removed J3: Screw_Terminal_01x06, TerminalBlock_Phoenix:TerminalBlock_Phoenix_MKDS-1,5-6_1x06_P5.00mm_Horizontal, symbol Connector:Screw_Terminal_01x06
- added MOD1: ~, SNES:ZD1006, symbol zd1006:ZD1006

Commit message: update
update
Parts:
- removed J1: Conn_02x10_Odd_Even, Connector_PinHeader_2.54mm:PinHeader_2x10_P2.54mm_Vertical, symbol Connector_Generic:Conn_02x10_Odd_Even
- removed R1, R10, R11, R12, R13, R14, R15, R16, R17, R18, R19, R2, R20, R21, R22, R23, R3, R4, R5, R6, R7, R8, R9: R, Resistor_SMD:R_0805_2012Metric_Pad1.20x1.40mm_HandSolder, symbol Device:R
- added C1: C0603_100nF_16V_X7R, Capacitor_SMD:C_0603_1608Metric, symbol Capacitors_SMD_0603:C0603_100nF_16V_X7R
- added F1, F10, F11, F12, F13, F14, F15, F16, F2, F3, F4, F5, F6, F7, F8, F9: Polyfuse, Fuse:Fuse_1812_4532Metric, symbol Device:Polyfuse
- added R1, R10, R11, R12, R13, R14, R15, R16, R2, R3, R4, R5, R6, R7, R8, R9: R0603_1k_1%_100mW_100PPM_AC, Resistor_SMD:R_0603_1608Metric, symbol Resistors_SMD_0603:R0603_1k_1%_100mW_100PPM_AC
- added U2: ESP32-DEVKITC-32UE, ESP32-DEVKITC-32UE:ESPRESSIF_ESP32-DEVKITC-32UE, symbol ESP32-DEVKITC-32UE:ESP32-DEVKITC-32UE
- MOD1: footprint SNES:ZD1006 -> ZD1006:ZD1006
- Q1, Q10, Q11, Q12, Q13, Q14, Q15, Q16, Q2, Q3, Q4, Q5, Q6, Q7, Q8, Q9: footprint Package_TO_SOT_THT:TO-251-3_Vertical -> Package_TO_SOT_SMD:TO-252-2
Connections:
- net LED0 is gone; now on net LED1: U1.6 (LED0)
- net +5V: now also C1.1
- net GND: now also MOD1.D1, MOD1.D4, MOD1.D7, C1.2
- net LED1: now also R1.1; no longer U1.7 (LED1)
- net LED10: now also U1.16 (LED9), R10.1; no longer U1.17 (LED10)
- net LED10_OUT: now also MOD1.B5, F10.2
- net LED11: now also U1.17 (LED10), R11.1; no longer U1.18 (LED11)
- net LED11_OUT: now also MOD1.B7, F11.2
- net LED12: now also U1.18 (LED11), R12.1; no longer U1.19 (LED12)
- net LED12_OUT: now also MOD1.B8, F12.2
- net LED13: now also U1.19 (LED12), R13.1; no longer U1.20 (LED13)
- net LED13_OUT: now also MOD1.C1, F13.2
- net LED14: now also U1.20 (LED13), R14.1; no longer U1.21 (LED14)
- net LED14_OUT: now also MOD1.C2, F14.2
- net LED15: now also U1.21 (LED14), R15.1; no longer U1.22 (LED15)
- net LED1_OUT: now also MOD1.A1, F1.2; no longer Q2.2 (D)
- net LED2: now also U1.7 (LED1), R2.1; no longer U1.8 (LED2)
- net LED2_OUT: now also MOD1.A2, F2.2; no longer Q3.2 (D)
- net LED3: now also U1.8 (LED2), R3.1; no longer U1.9 (LED3)
- net LED3_OUT: now also MOD1.A4, F3.2; no longer Q4.2 (D)
- net LED4: now also U1.9 (LED3), R4.1; no longer U1.10 (LED4)
- net LED4_OUT: now also MOD1.A5, F4.2; no longer Q5.2 (D)
- net LED5: now also U1.10 (LED4), R5.1; no longer U1.11 (LED5)
- net LED5_OUT: now also MOD1.A7, F5.2
- net LED6: now also U1.11 (LED5), R6.1; no longer U1.12 (LED6)
- net LED6_OUT: now also MOD1.A8, F6.2
- net LED7: now also U1.12 (LED6), R7.1; no longer U1.13 (LED7)
- net LED7_OUT: now also MOD1.B1, F7.2
- net LED8: now also U1.13 (LED7), R8.1; no longer U1.15 (LED8)
- net LED8_OUT: now also MOD1.B2, F8.2
- net LED9: now also U1.15 (LED8), R9.1; no longer U1.16 (LED9)
- net LED9_OUT: now also MOD1.B4, F9.2
- net at Q1.1 (G): now also R1.2
- net at Q8.1 (G): now also R8.2
- net at Q2.1 (G): now also R2.2
- net at Q3.1 (G): now also R3.2
- net at Q4.1 (G): now also R4.2
- net at Q7.1 (G): now also R7.2
- net at Q5.1 (G): now also R5.2
- net at Q6.1 (G): now also R6.2
- net at Q6.2 (D): now also F6.1
- net at Q7.2 (D): now also F7.1
- net at Q8.2 (D): now also F8.1
- net at Q16.1 (G): now also R16.2
- net at Q16.2 (D): now also F16.1
- net at Q15.1 (G): now also R15.2
- net at Q15.2 (D): now also F15.1
- net at Q14.1 (G): now also R14.2
- net at Q14.2 (D): now also F14.1
- net at Q13.1 (G): now also R13.2
- net at Q13.2 (D): now also F13.1
- net at Q12.1 (G): now also R12.2
- net at Q12.2 (D): now also F12.1
- net at Q11.1 (G): now also R11.2
- net at Q11.2 (D): now also F11.1
- net at Q10.1 (G): now also R10.2
- net at Q10.2 (D): now also F10.1
- net at Q9.1 (G): now also R9.2
- net at Q9.2 (D): now also F9.1
- net VBUS: now reaches MOD1.A3
- net VBUS: now also MOD1.A6, MOD1.B3, MOD1.B6, MOD1.C3, MOD1.C6, MOD1.D3, MOD1.D6, MOD1.D8
- net LED0_OUT: no longer names the net of Q1.2 (D)
- net LED0_OUT: now also F1.1
- new net: F2.1, Q2.2 (D)
- new net: F3.1, Q3.2 (D)
- new net: F4.1, Q4.2 (D)
- new net: F5.1, Q5.2 (D)
- new net LED15_OUT: F15.2, MOD1.C4
- new net LED16: R16.1, U1.22 (LED15)
- new net LED16_OUT: F16.2, MOD1.C5
- new net LED17_OUT: MOD1.C7
- new net LED18_OUT: MOD1.C8
Other:
- note added: "1812L050ZR"
- moved on the sheet: MOD1B, MOD1C, MOD1D, Q1, Q10, Q11, Q12, Q13, Q14, Q15, Q16, Q2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

Commit message: update
Parts:
- added Q17, Q18: BSS138, Package_TO_SOT_SMD:SOT-23, symbol Transistor_FET:BSS138
- added R17, R18, R19, R20, R21: R0603_10k_1%_100mW_100PPM_AC, Resistor_SMD:R_0603_1608Metric, symbol Resistors_SMD_0603:R0603_10k_1%_100mW_100PPM_AC
- added U4: Mini360, Mini360_step-down:Mini360_step-down, symbol mini360:Mini360
Connections:
- net +5V: now also U2.19 (5V), R18.1, R21.1, U4.4 (OUT+)
- net GND: now also U2.14 (GND), U2.20 (GND__1), U2.26 (GND__2), U4.1 (IN-), U4.3 (OUT-)
- net VBUS: now also U4.2 (IN+)
- net nOE: now also U2.21 (23)
- net +3.3V: now reaches U2.1 (3V3)
- net +3.3V: now also Q17.1 (G), Q18.1 (G), R17.2, R19.1, R20.1
- net at U2.2 (EN): now also R17.1
- net SCL_L: now reaches U2.22
- net SCL_L: now also Q17.2 (S), R19.2
- net SDA_L: now reaches U2.25 (21)
- net SDA_L: now also Q18.2 (S), R20.2
- net SCL renamed SCL_H
- net SCL_H: now also Q17.3 (D), R18.2
- net SDA renamed SDA_H
- net SDA_H: now also Q18.3 (D), R21.2
Other:
- company: (none) -> JKBI
- title: (none) -> Stairs LED controller

Commit message: update
Parts:
- added JP1, JP2, JP3: SolderJumper_3_Open, Jumper:SolderJumper-3_P1.3mm_Open_RoundedPad1.0x1.5mm_NumberLabels, symbol Jumper:SolderJumper_3_Open
Connections:
- net +5V: now also JP1.3 (B), JP2.3 (B), JP3.3 (B)
- net GND: now also U1.24 (A5), U1.25 (A6), U1.4 (A3), U1.5 (A4), JP1.1 (A), JP2.1 (A), JP3.1 (A)
- net A0: now reaches U1.1 (A0)
- net A0: now also JP1.2 (C)
- net A1: now reaches U1.2 (A1)
- net A1: now also JP2.2 (C)
- net A2: now reaches U1.3 (A2)
- net A2: now also JP3.2 (C)

Commit message: UPDATE
Parts:
- removed U4: Mini360, Mini360_step-down:Mini360_step-down, symbol mini360:Mini360
- added J1: Conn_01x04_Pin, Connector_PinHeader_2.54mm:PinHeader_1x04_P2.54mm_Vertical, symbol 380-015-113L001:Conn_01x04_Pin
- added R22, R23, R26, R27: R0603_4.7k_1%_100mW_100PPM_AC, Resistor_SMD:R_0603_1608Metric, symbol Resistors_SMD_0603:R0603_4.7k_1%_100mW_100PPM_AC
- added R24, R25, R28, R29: R0805_3.01k_1%_125mW_100PPM_RC, Resistor_SMD:R_0805_2012Metric, symbol Resistors_SMD_0805:R0805_3.01k_1%_125mW_100PPM_RC
- added U3, U5, U6, U7: PC817, Package_DIP:DIP-4_W7.62mm, symbol Isolator:PC817
- added U8: R-78E5.0-1.0, Converter_DCDC:Converter_DCDC_RECOM_R-78E-0.5_THT, symbol Regulator_Switching:R-78E5.0-1.0
Connections:
- net +3.3V: now also R22.1, R23.1, R26.1, R27.1
- net +5V: now also J1.1 (Pin_1), U8.3 (OUT)
- net GND: now also J1.4 (Pin_4), U3.2, U3.3, U5.2, U5.3, U6.2, U6.3, U7.2, U7.3, U8.2 (GND)
- net SCL_H: now also J1.3 (Pin_3)
- net SDA_H: now also J1.2 (Pin_2)
- net VBUS: now also U8.1 (IN)
- net IN4_L: now reaches U2.27 (19)
- net IN4_L: now also R27.2, U7.4
- net IN3_L: now reaches U2.28 (18)
- net IN3_L: now also R26.2, U6.4
- net IN2_L: now reaches U2.29 (5)
- net IN2_L: now also R23.2, U5.4
- net IN1_L: now reaches U2.30 (17)
- net IN1_L: now also R22.2, U3.4
- net IN1_H: now reaches MOD1.D2
- net IN1_H: now also R24.1
- net IN2_H: now reaches MOD1.D5
- net IN2_H: now also R25.1
- new net: R25.2, U5.1
- new net: R24.2, U3.1
- new net: R29.2, U7.1
- new net: R28.2, U6.1
- new net IN3_H: R28.1
- new net IN4_H: R29.1
Other:
- moved on the sheet: MOD1D, R17, U2

Commit message: update
Parts:
- added C2: C0603_100nF_16V_X7R, Capacitor_SMD:C_0603_1608Metric, symbol Capacitors_SMD_0603:C0603_100nF_16V_X7R
- added F17: Polyfuse, Fuse:Fuse_1812_4532Metric, symbol Device:Polyfuse
- added J2: Conn_01x04_Pin, Connector_PinHeader_2.54mm:PinHeader_1x04_P2.54mm_Vertical, symbol Connector:Conn_01x04_Pin
- added J3: Conn_01x04_Pin, Connector_PinHeader_2.54mm:PinHeader_1x04_P2.54mm_Horizontal, symbol Connector:Conn_01x04_Pin
- added Q19: BSS138, Package_TO_SOT_SMD:SOT-23, symbol Transistor_FET:BSS138
- added R30, R31, R32: R0603_4.7k_1%_100mW_100PPM_AC, Resistor_SMD:R_0603_1608Metric, symbol Resistors_SMD_0603:R0603_4.7k_1%_100mW_100PPM_AC
- added U4: MCP23008-xSO, Package_SO:SOIC-18W_7.5x11.6mm_P1.27mm, symbol Interface_Expansion:MCP23008-xSO
- J1: value Conn_01x04_Pin -> Conn_01x04_Socket; footprint Connector_PinHeader_2.54mm:PinHeader_1x04_P2.54mm_Vertical -> Connector_PinSocket_2.54mm:PinSocket_1x04_P2.54mm_Horizontal; symbol 380-015-113L001:Conn_01x04_Pin -> Connector:Conn_01x04_Socket
Connections:
- net LED17_OUT is gone; now on net IN4_H: MOD1.C7
- net LED18_OUT is gone; now on net IN3_H: MOD1.C8
- net +3.3V: now also J2.1 (Pin_1)
- net +5V: now also C2.2, J3.1 (Pin_1), R30.1, R31.1, R32.1, U4.18 (VDD), U4.6 (~{RESET})
- net GND: now also C2.1, J2.4 (Pin_4), J3.4 (Pin_4), Q19.2 (S), U4.3 (A2), U4.4 (A1), U4.5 (A0), U4.9 (VSS)
- net IN2_L: now also U2.32 (4); no longer U2.29 (5)
- net SCL_H: now also J3.3 (Pin_3), R31.2, U4.1 (SCL)
- net SCL_L: now also J2.3 (Pin_3)
- net SDA_H: now also J3.2 (Pin_2), R30.2, U4.2 (SDA)
- net SDA_L: now also J2.2 (Pin_2)
- net VBUS: now also F17.1; no longer U8.1 (IN)
- net nOE: now also Q19.3 (D), R32.2; no longer U2.21 (23)
- new net: F17.2, U8.1 (IN)
- new net INT_H: U4.8 (INT)
- new net OE: Q19.1 (G), U2.21 (23)
- no-connect marks 0 -> 25
Other:
- moved on the sheet: Q17, Q18, R18, R19, R20, R21
