File: hardware/led_stairs_controller.kicad_sch (KiCad schematic)
At the start: 85 parts, among them J1 Conn_01x04_Socket, J2 Conn_01x04_Pin, J3 Conn_01x04_Pin, Q1 QM6006D, Q10 QM6006D, Q11 QM6006D, Q12 QM6006D, Q13 QM6006D, Q14 QM6006D, Q15 QM6006D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

Commit message: update
Parts:
- added C3: C0603_100nF_16V_X7R, Capacitor_SMD:C_0603_1608Metric, symbol Capacitors_SMD_0603:C0603_100nF_16V_X7R
- J1: value Conn_01x04_Socket -> Conn_01x05_Socket; symbol Connector:Conn_01x04_Socket -> Connector:Conn_01x05_Socket
Connections:
- net +3.3V: no longer R22.1, R23.1, R26.1, R27.1
- net +5V: now also C3.2
- net A0: now also U4.5 (A0)
- net A1: now also U4.4 (A1)
- net A2: now also U4.3 (A2)
- net GND: now also J1.5 (Pin_5), C3.1; no longer J1.4 (Pin_4), U4.3 (A2), U4.4 (A1), U4.5 (A0)
- net IN1_L: now also U2.32 (4), U4.13 (GP3); no longer U2.30 (17)
- net IN2_L: now also U2.30 (17), U4.12 (GP2); no longer U2.32 (4)
- net IN3_L: now also U4.11 (GP1)
- net IN4_L: now also U4.10 (GP0)
- net nOE: now also U4.14 (GP4)
- new net P-UP: R22.1, R23.1, R26.1, R27.1
Other:
- moved on the sheet: R30, R31

Commit message: update
Parts:
- added R33: R0603_4.7k_1%_100mW_100PPM_AC, Resistor_SMD:R_0603_1608Metric, symbol Resistors_SMD_0603:R0603_4.7k_1%_100mW_100PPM_AC
- J1: footprint Connector_PinSocket_2.54mm:PinSocket_1x04_P2.54mm_Horizontal -> Connector_PinSocket_2.54mm:PinSocket_1x05_P2.54mm_Horizontal
- J3: value Conn_01x04_Pin -> Conn_01x05_Pin; footprint Connector_PinHeader_2.54mm:PinHeader_1x04_P2.54mm_Horizontal -> Connector_PinHeader_2.54mm:PinHeader_1x05_P2.54mm_Horizontal; symbol Connector:Conn_01x04_Pin -> Connector:Conn_01x05_Pin
Connections:
- net +5V: now also R33.1
- net GND: now also J3.5 (Pin_5); no longer J3.4 (Pin_4)
- net INT_H: now also J1.4 (Pin_4), J3.4 (Pin_4), R33.2

Commit message: update
Parts:
- added Q20: BSS138, Package_TO_SOT_SMD:SOT-23, symbol Transistor_FET:BSS138
- added R34, R35: R0603_10k_1%_100mW_100PPM_AC, Resistor_SMD:R_0603_1608Metric, symbol Resistors_SMD_0603:R0603_10k_1%_100mW_100PPM_AC
- J2: value Conn_01x04_Pin -> Conn_01x05_Pin; footprint Connector_PinHeader_2.54mm:PinHeader_1x04_P2.54mm_Vertical -> Connector_PinHeader_2.54mm:PinHeader_1x05_P2.54mm_Vertical; symbol Connector:Conn_01x04_Pin -> Connector:Conn_01x05_Pin
Connections:
- net +3.3V: now also Q20.1 (G), R34.1
- net +5V: now also R35.1
- net GND: now also J2.5 (Pin_5); no longer J2.4 (Pin_4)
- net INT_H: now also Q20.3 (D), R35.2
- new net INT_L: J2.4 (Pin_4), Q20.2 (S), R34.2
Other:
- moved on the sheet: Q17, Q18, R18, R19, R20, R21

Commit message: update
Parts:
- removed R24, R28, R29: R0805_3.01k_1%_125mW_100PPM_RC, Resistor_SMD:R_0805_2012Metric, symbol Resistors_SMD_0805:R0805_3.01k_1%_125mW_100PPM_RC
- added JP4: SolderJumper_3_Open, Jumper:SolderJumper-3_P1.3mm_Open_RoundedPad1.0x1.5mm_NumberLabels, symbol Jumper:SolderJumper_3_Open
- added R24, R28, R29, R36, R37, R38, R39: R0805_1.5k_1%_125mW_100PPM_AC, Resistor_SMD:R_0805_2012Metric, symbol Resistors_SMD_0805:R0805_1.5k_1%_125mW_100PPM_AC
- R25: value R0805_3.01k_1%_125mW_100PPM_RC -> R0805_1.5k_1%_125mW_100PPM_AC; symbol Resistors_SMD_0805:R0805_3.01k_1%_125mW_100PPM_RC -> Resistors_SMD_0805:R0805_1.5k_1%_125mW_100PPM_AC; Description_1 RES SMD 3.01K OHM 1% 1/8W 0805 -> RES SMD 1.5K OHM 1% 1/8W 0805; Manufacturer Part Number RC0805FR-073K01L -> AC0805FR-071K5L; Supplier Part Number 311-3.01KCRCT-ND -> YAG3701CT-ND; Value1 3.01k -> 1.5k
Connections:
- net +3.3V: now also JP4.1 (A)
- net +5V: now also JP4.3 (B)
- net GND: now also R36.1, R37.1, R38.1, R39.1; no longer U3.2, U5.2, U6.2, U7.2
- net IN1_H: now also R24.1
- net IN3_H: now also R28.1
- net IN4_H: now also R29.1
- net P-UP: now also JP4.2 (C)
- net at U3.1: now also R24.2
- net at U7.1: now also R29.2
- net at U6.1: now also R28.2
- new net: R36.2, U5.2
- new net: R38.2, U6.2
- new net: R39.2, U7.2
- new net: R37.2, U3.2
Other:
- moved on the sheet: R25

Commit message: update
Parts:
- added C4, C5: C0603_100nF_16V_X7R, Capacitor_SMD:C_0603_1608Metric, symbol Capacitors_SMD_0603:C0603_100nF_16V_X7R
- added C6: C1210_10µF_50V_X5R, Capacitor_SMD:C_1210_3225Metric, symbol Capacitors_SMD_1210:C1210_10µF_50V_X5R
- added C7: C1210_100µF_16V_X5R, Capacitor_SMD:C_1210_3225Metric, symbol Capacitors_SMD_1210:C1210_100µF_16V_X5R
- added JP5, JP6, JP7, JP8: Jumper_2_Open, Jumper:SolderJumper-2_P1.3mm_Open_RoundedPad1.0x1.5mm, symbol Jumper:Jumper_2_Open
Connections:
- net +3.3V: now also C4.1
- net +5V: now also C5.1, C7.1
- net GND: now also C4.2, C5.2, C6.2, C7.2
- net IN1_L: now also JP5.1 (A); no longer U2.32 (4)
- net IN2_L: now also JP6.1 (A); no longer U2.30 (17)
- net IN3_L: now also JP7.1 (A); no longer U2.28 (18)
- net IN4_L: now also JP8.2 (B); no longer U2.27 (19)
- net at F17.2, U8.1 (IN): now also C6.1
- new net: JP8.1 (A), U2.27 (19)
- new net: JP7.2 (B), U2.28 (18)
- new net: JP6.2 (B), U2.30 (17)
- new net: JP5.2 (B), U2.32 (4)
Other:
- moved on the sheet: C2
