File: hardware/led_stairs_controller.kicad_sch (KiCad schematic)
At the start: 103 parts, among them J1 Conn_01x05_Socket, J2 Conn_01x05_Pin, J3 Conn_01x05_Pin, Q1 QM6006D, Q10 QM6006D, Q11 QM6006D, Q12 QM6006D, Q13 QM6006D, Q14 QM6006D, Q15 QM6006D, Q16 QM6006D, Q17 BSS138, Q18 BSS138, Q19 BSS138, Q2 QM6006D, Q20 BSS138, Q3 QM6006D, Q4 QM6006D, Q5 QM6006D, Q6 QM6006D, Q7 QM6006D, Q8 QM6006D, Q9 QM6006D, U1 PCA9635, U2 ESP32-DEVKITC-32UE, U3 PC817, U4 MCP23008-xSO, U5 PC817, U6 PC817, U7 PC817, U8 R-78E5.0-1.0

Commit message: update
Parts:
- removed Q1, Q10, Q11, Q12, Q13, Q14, Q15, Q16, Q2, Q3, Q4, Q5, Q6, Q7, Q8, Q9: QM6006D, Package_TO_SOT_SMD:TO-252-2, symbol Transistor_FET:QM6006D
- added C8, C9: C0603_100nF_16V_X7R, Capacitor_SMD:C_0603_1608Metric, symbol Capacitors_SMD_0603:C0603_100nF_16V_X7R
- added J1, J11: DIN41612_02x32_AC, Connector_DIN:DIN41612_C_2x32_Male_Horizontal_THT, symbol Connector:DIN41612_02x32_AC
- added Q1, Q10, Q11, Q12, Q13, Q14, Q15, Q16, Q2, Q3, Q4, Q5, Q6, Q7, Q8, Q9: IRF7341PBF, Package_SO:SOIC-8_3.9x4.9mm_P1.27mm, symbol Transistor_FET:IRF7341PBF
- added R40, R41, R42, R43, R44, R45, R46, R47, R48, R49, R50, R51, R52, R53, R54, R55: R0603_4.7k_1%_100mW_100PPM_AC, Resistor_SMD:R_0603_1608Metric, symbol Resistors_SMD_0603:R0603_4.7k_1%_100mW_100PPM_AC
- added R56, R57, R58, R59, R60, R61, R62, R63, R64, R65, R66, R67, R68, R69, R70, R71: R0603_1k_1%_100mW_100PPM_AC, Resistor_SMD:R_0603_1608Metric, symbol Resistors_SMD_0603:R0603_1k_1%_100mW_100PPM_AC
- added U10: PCA9635, Package_SO:TSSOP-28_4.4x9.7mm_P0.65mm, symbol Driver_LED:PCA9635
- added U9: CD74HC4067M, Package_SO:SOIC-24W_7.5x15.4mm_P1.27mm, symbol 74xx:CD74HC4067M
- renumbered J1 to J17, J3 to J18, J2 to J19
Connections:
- net +5V: now also C8.2, C9.1, U10.28 (VDD), U10.4 (A3), U9.24 (VCC)
- net A0: now also U10.1 (A0)
- net A1: now also U10.2 (A1)
- net A2: now also U10.3 (A2)
- net GND: now also C8.1, C9.2, J1.a13 (Pin_a13), J1.a19 (Pin_a19), J1.a25 (Pin_a25), J1.a31 (Pin_a31), J1.c13 (Pin_c13), J1.c19 (Pin_c19), J1.c25 (Pin_c25), J1.c31 (Pin_c31), J11.a13 (Pin_a13), J11.a19 (Pin_a19), J11.a25 (Pin_a25), J11.a31 (Pin_a31), J11.a7 (Pin_a7), J11.c13 (Pin_c13), J11.c19 (Pin_c19), J11.c25 (Pin_c25), J11.c31 (Pin_c31), J11.c7 (Pin_c7), Q1.1 (S1), Q1.3 (S2), Q10.1 (S1), Q10.3 (S2), Q11.1 (S1), Q11.3 (S2), Q12.1 (S1), Q12.3 (S2), Q13.1 (S1), Q13.3 (S2), Q14.1 (S1), Q14.3 (S2), Q15.1 (S1), Q15.3 (S2), Q16.1 (S1), Q16.3 (S2), Q2.1 (S1), Q2.3 (S2), Q3.1 (S1), Q3.3 (S2), Q4.1 (S1), Q4.3 (S2), Q5.1 (S1), Q5.3 (S2), Q6.1 (S1), Q6.3 (S2), Q7.1 (S1), Q7.3 (S2), Q8.1 (S1), Q8.3 (S2), Q9.1 (S1), Q9.3 (S2), U10.14 (VSS), U10.24 (A5), U10.25 (A6), U10.5 (A4), U9.12 (GND)
- net LED10_OUT: no longer F10.2
- net LED11_OUT: no longer F11.2
- net LED12_OUT: no longer F12.2
- net LED13_OUT: no longer F13.2
- net LED14_OUT: no longer F14.2
- net LED15_OUT: no longer F15.2
- net LED16_OUT: no longer F16.2
- net LED1_OUT: no longer F1.2
- net LED2_OUT: no longer F2.2
- net LED3_OUT: no longer F3.2
- net LED4_OUT: no longer F4.2
- net LED5_OUT: no longer F5.2
- net LED6_OUT: no longer F6.2
- net LED7_OUT: no longer F7.2
- net LED8_OUT: no longer F8.2
- net LED9_OUT: no longer F9.2
- net SCL_H: now also U10.26 (SCL)
- net SDA_H: now also U10.27 (SDA)
- net VBUS: now also F1.1, F10.1, F11.1, F12.1, F13.1, F14.1, F15.1, F16.1, F2.1, F3.1, F4.1, F5.1, F6.1, F7.1, F8.1, F9.1
- net nOE: now also U10.23 (~{OE})
- net at R1.2: now also Q1.2 (G1)
- net at R2.2: now also Q2.2 (G1)
- net at R3.2: now also Q3.2 (G1)
- net at R4.2: now also Q4.2 (G1)
- net at R5.2: now also Q5.2 (G1)
- net at R6.2: now also Q6.2 (G1)
- net at R7.2: now also Q7.2 (G1)
- net at R8.2: now also Q8.2 (G1)
- net at R16.2: now also Q16.2 (G1)
- net at R15.2: now also Q15.2 (G1)
- net at R14.2: now also Q14.2 (G1)
- net at R13.2: now also Q13.2 (G1)
- net at R12.2: now also Q12.2 (G1)
- net at R11.2: now also Q11.2 (G1)
- net at R10.2: now also Q10.2 (G1)
- net at R9.2: now also Q9.2 (G1)
- net LED1 renamed LEDA1
- net LED10 renamed LEDA10
- net LED11 renamed LEDA11
- net LED12 renamed LEDA12
- net LED13 renamed LEDA13
- net LED14 renamed LEDA14
- net LED15 renamed LEDA15
- net LED16 renamed LEDA16
- net LED2 renamed LEDA2
- net LED3 renamed LEDA3
- net LED4 renamed LEDA4
- net LED5 renamed LEDA5
- net LED6 renamed LEDA6
- net LED7 renamed LEDA7
- net LED8 renamed LEDA8
- net LED9 renamed LEDA9
- new net: Q2.4 (G2), R57.2
- new net: R42.1, U9.6 (I3)
- new net: F11.2, J1.a26 (Pin_a26)
- new net: Q8.4 (G2), R63.2
- new net: Q7.4 (G2), R62.2
- new net: F15.2, J1.c26 (Pin_c26)
- new net: F1.2, J11.a2 (Pin_a2)
- new net: R52.1, U9.22 (I9)
- new net: R49.1, U9.17 (I14)
- new net: R46.1, U9.23 (I8)
- new net: R44.1, U9.5 (I4)
- new net: F2.2, J11.a8 (Pin_a8)
- new net: R48.1, U9.19 (I12)
- new net: R43.1, U9.7 (I2)
- new net: R53.1, U9.20 (I11)
- new net: Q3.4 (G2), R58.2
- new net: Q16.4 (G2), R71.2
- new net: R40.1, U9.9 (I0)
- new net: F7.2, J11.c8 (Pin_c8)
- new net: F10.2, J11.c26 (Pin_c26)
- new net: F6.2, J11.c2 (Pin_c2)
- new net: Q15.4 (G2), R70.2
- new net: R51.1, U9.2 (I7)
- new net: F13.2, J1.a14 (Pin_a14)
- new net: F12.2, J1.a20 (Pin_a20)
- new net: F16.2, J1.c14 (Pin_c14)
- new net: F14.2, J1.c20 (Pin_c20)
- new net: R55.1, U9.16 (I15)
- new net: R50.1, U9.4 (I5)
- new net: F5.2, J11.a26 (Pin_a26)
- new net: Q10.4 (G2), R65.2
- new net: F3.2, J11.a14 (Pin_a14)
- new net: Q11.4 (G2), R66.2
- new net: F9.2, J11.c20 (Pin_c20)
- new net: Q4.4 (G2), R59.2
- new net: Q12.4 (G2), R67.2
- new net: R41.1, U9.8 (I1)
- new net: Q14.4 (G2), R69.2
- new net: Q6.4 (G2), R61.2
- new net: Q1.4 (G2), R56.2
- new net: F4.2, J11.a20 (Pin_a20)
- new net: F8.2, J11.c14 (Pin_c14)
- new net: R45.1, U9.3 (I6)
- new net: Q13.4 (G2), R68.2
- new net: R54.1, U9.18 (I13)
- new net: R47.1, U9.21 (I10)
- new net: Q9.4 (G2), R64.2
- new net: Q5.4 (G2), R60.2
- new net LED10A_OUT: J11.c28 (Pin_c28), Q10.7 (D1), Q10.8 (D1)
- new net LED10B_OUT: J11.c29 (Pin_c29), Q10.5 (D2), Q10.6 (D2)
- new net LED11A_OUT: J1.a28 (Pin_a28), Q11.7 (D1), Q11.8 (D1)
- new net LED11B_OUT: J1.a29 (Pin_a29), Q11.5 (D2), Q11.6 (D2)
- new net LED12A_OUT: J1.a22 (Pin_a22), Q12.5 (D2), Q12.6 (D2), Q12.7 (D1), Q12.8 (D1)
- new net LED12B_OUT: J1.a23 (Pin_a23)
- new net LED13A_OUT: J1.a16 (Pin_a16), Q13.7 (D1), Q13.8 (D1)
- new net LED13B_OUT: Q13.5 (D2), Q13.6 (D2)
- new net LED14A_OUT: J1.c22 (Pin_c22), Q14.7 (D1), Q14.8 (D1)
- new net LED14B_OUT: J1.c23 (Pin_c23), Q14.5 (D2), Q14.6 (D2)
- new net LED15A_OUT: J1.c28 (Pin_c28), Q15.7 (D1), Q15.8 (D1)
- new net LED15B_OUT: J1.c29 (Pin_c29), Q15.5 (D2), Q15.6 (D2)
- new net LED16A_OUT: J1.c16 (Pin_c16), Q16.7 (D1), Q16.8 (D1)
- new net LED16B_OUT: J1.c17 (Pin_c17), Q16.5 (D2), Q16.6 (D2)
- new net LED1A_OUT: J11.a4 (Pin_a4), Q1.7 (D1), Q1.8 (D1)
- new net LED1B_OUT: J11.a5 (Pin_a5), Q1.5 (D2), Q1.6 (D2)
- new net LED2A_OUT: J11.a10 (Pin_a10), Q2.7 (D1), Q2.8 (D1)
- new net LED2B_OUT: J11.a11 (Pin_a11), Q2.5 (D2), Q2.6 (D2)
- new net LED3A_OUT: J11.a16 (Pin_a16), Q3.7 (D1), Q3.8 (D1)
- new net LED3B_OUT: J1.a17 (Pin_a17), J11.a17 (Pin_a17), Q3.5 (D2), Q3.6 (D2)
- new net LED4A_OUT: J11.a22 (Pin_a22), Q4.7 (D1), Q4.8 (D1)
- new net LED4B_OUT: J11.a23 (Pin_a23), Q4.5 (D2), Q4.6 (D2)
- new net LED5A_OUT: J11.a28 (Pin_a28), Q5.7 (D1), Q5.8 (D1)
- new net LED5B_OUT: J11.a29 (Pin_a29), Q5.5 (D2), Q5.6 (D2)
- new net LED6A_OUT: J11.c4 (Pin_c4), Q6.7 (D1), Q6.8 (D1)
- new net LED6B_OUT: J11.c5 (Pin_c5), Q6.5 (D2), Q6.6 (D2)
- new net LED7A_OUT: J11.c10 (Pin_c10), Q7.7 (D1), Q7.8 (D1)
- new net LED7B_OUT: J11.c11 (Pin_c11), Q7.5 (D2), Q7.6 (D2)
- new net LED8A_OUT: J11.c16 (Pin_c16), Q8.7 (D1), Q8.8 (D1)
- new net LED8B_OUT: J11.c17 (Pin_c17), Q8.5 (D2), Q8.6 (D2)
- new net LED9A_OUT: J11.c22 (Pin_c22), Q9.7 (D1), Q9.8 (D1)
- new net LED9B_OUT: J11.c23 (Pin_c23), Q9.5 (D2), Q9.6 (D2)
- new net LEDB1: R56.1, U10.6 (LED0)
- new net LEDB10: R65.1, U10.16 (LED9)
- new net LEDB11: R66.1, U10.17 (LED10)
- new net LEDB12: R67.1, U10.18 (LED11)
- new net LEDB13: R68.1, U10.19 (LED12)
- new net LEDB14: R69.1, U10.20 (LED13)
- new net LEDB15: R70.1, U10.21 (LED14)
- new net LEDB16: R71.1, U10.22 (LED15)
- new net LEDB2: R57.1, U10.7 (LED1)
- new net LEDB3: R58.1, U10.8 (LED2)
- new net LEDB4: R59.1, U10.9 (LED3)
- new net LEDB5: R60.1, U10.10 (LED4)
- new net LEDB6: R61.1, U10.11 (LED5)
- new net LEDB7: R62.1, U10.12 (LED6)
- new net LEDB8: R63.1, U10.13 (LED7)
- new net LEDB9: R64.1, U10.15 (LED8)
- new net WS2811: U9.1 (COM)
- new net WS2811_1: J11.a3 (Pin_a3), R40.2
- new net WS2811_10: J11.c27 (Pin_c27), R52.2
- new net WS2811_11: J1.a27 (Pin_a27), R47.2
- new net WS2811_12: J1.a21 (Pin_a21), R53.2
- new net WS2811_13: J1.a15 (Pin_a15), R48.2
- new net WS2811_14: J1.c21 (Pin_c21), R54.2
- new net WS2811_15: J1.c27 (Pin_c27), R49.2
- new net WS2811_16: J1.c15 (Pin_c15), R55.2
- new net WS2811_2: J11.a9 (Pin_a9), R41.2
- new net WS2811_3: J11.a15 (Pin_a15), R43.2
- new net WS2811_4: J11.a21 (Pin_a21), R42.2
- new net WS2811_5: J11.a27 (Pin_a27), R44.2
- new net WS2811_6: J11.c3 (Pin_c3), R50.2
- new net WS2811_7: J11.c9 (Pin_c9), R45.2
- new net WS2811_8: J11.c15 (Pin_c15), R51.2
- new net WS2811_9: J11.c21 (Pin_c21), R46.2
Other:
- moved on the sheet: C1, C2, C3, C6, C7, F17, J19, JP4, MOD1A, MOD1B, MOD1C, MOD1D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

Commit message: update
Connections:
- net LED12A_OUT: no longer Q12.5 (D2), Q12.6 (D2)
- net LED12B_OUT: now also Q12.5 (D2), Q12.6 (D2)
- net LED13B_OUT: now also J1.a17 (Pin_a17)
- net LED3B_OUT: no longer J1.a17 (Pin_a17)
Changed lines of the file:
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@@
 		)
 	)
-	(label "LED12A_OUT"
+	(label "LED12B_OUT"
 		(at 367.665 234.95 180)
 		(effects
@@
 		)
 	)
-	(label "LED3B_OUT"
+	(label "LED13B_OUT"
 		(at 421.64 74.295 0)
 		(effects

Commit message: update
Connections:
- net GND: now also J1.a7 (Pin_a7), J1.c7 (Pin_c7)
- net VBUS: now also J1.a2 (Pin_a2), J1.c2 (Pin_c2)
Changed lines of the file:
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@@
 	)
 	(junction
+		(at 486.41 36.195)
+		(diameter 0)
+		(color 0 0 0 0)
+	)
+	(junction
 		(at 528.32 185.42)
 		(diameter 0)
@@
 	)
 	(junction
+		(at 461.01 64.135)
+		(diameter 0)
+		(color 0 0 0 0)
+	)
+	(junction
+		(at 417.83 36.195)
+		(diameter 0)
+		(color 0 0 0 0)
+	)
+	(junction
 		(at 502.285 66.675)
 		(diameter 0)
@@
 	)
 	(junction
+		(at 443.23 64.135)
+		(diameter 0)
+		(color 0 0 0 0)
+	)
+	(junction
 		(at 527.685 94.615)
 		(diameter 0)
@@
 	(wire
 		(pts
+			(xy 445.77 48.895) (xy 443.23 48.895)
+		)
+		(stroke
+			(width 0)
+			(type default)
+		)
+	)
+	(wire
+		(pts
 			(xy 570.865 51.435) (xy 570.865 66.675)
 		)
@@
 	(wire
 		(pts
+			(xy 461.01 48.895) (xy 461.01 64.135)
+		)
+		(stroke
+			(width 0)
+			(type default)
+		)
+	)
+	(wire
+		(pts
 			(xy 238.76 153.67) (xy 252.73 153.67)
 		)
@@
 	(wire
 		(pts
+			(xy 458.47 36.195) (xy 486.41 36.195)
+		)
+		(stroke
+			(width 0)
+			(type default)
+		)
+	)
+	(wire
+		(pts
 			(xy 121.92 316.23) (xy 116.84 316.23)
 		)
@@
 	(wire
 		(pts
+			(xy 417.83 36.195) (xy 445.77 36.195)
+		)
+		(stroke
+			(width 0)
+			(type default)
+		)
+	)
+	(wire
+		(pts
 			(xy 45.72 20.32) (xy 45.72 22.86)
 		)
@@
 	(wire
 		(pts
+			(xy 486.41 36.195) (xy 486.41 66.675)
+		)
+		(stroke
+			(width 0)
+			(type default)
+		)
+	)
+	(wire
+		(pts
 			(xy 238.76 163.83) (xy 252.73 163.83)
 		)
@@
 	(wire
 		(pts
+			(xy 417.83 36.195) (xy 417.83 66.675)
+		)
+		(stroke
+			(width 0)
+			(type default)
+		)
+	)
+	(wire
+		(pts
 			(xy 35.56 382.27) (xy 35.56 387.35)
 		)
@@
 	(wire
 		(pts
-			(xy 486.41 61.595) (xy 486.41 66.675)
+			(xy 486.41 31.115) (xy 486.41 36.195)
 		)
 		(stroke
@@
 	(wire
 		(pts
+			(xy 443.23 48.895) (xy 443.23 64.135)
+		)
+		(stroke
+			(width 0)
+			(type default)
+		)
+	)
+	(wire
+		(pts
 			(xy 238.76 173.99) (xy 252.73 173.99)
 		)
@@
 	(wire
 		(pts
+			(xy 458.47 48.895) (xy 461.01 48.895)
+		)
+		(stroke
+			(width 0)
+			(type default)
+		)
+	)
+	(wire
+		(pts
 			(xy 421.64 86.995) (xy 445.77 86.995)
 		)
@@
 	(wire
 		(pts
-			(xy 417.83 60.96) (xy 417.83 66.675)
+			(xy 417.83 31.115) (xy 417.83 36.195)
 		)
 		(stroke
@@
 	(symbol
 		(lib_id "power:VBUS")
-		(at 486.41 61.595 0)
+		(at 486.41 31.115 0)
 		(unit 1)
 		(exclude_from_sim no)
@@
 		(dnp no)
 		(property "Reference" "#PWR077"
-			(at 486.41 65.405 0)
+			(at 486.41 34.925 0)
 			(effects
 				(font
@@
 		)
 		(property "Value" "VBUS"
-			(at 486.41 57.15 0)
+			(at 486.41 26.67 0)
 			(effects
 				(font
@@
 		)
 		(property "Footprint" ""
-			(at 486.41 61.595 0)
+			(at 486.41 31.115 0)
 			(effects
 				(font
@@
 		)
 		(property "Datasheet" ""
-			(at 486.41 61.595 0)
+			(at 486.41 31.115 0)
 			(effects
 				(font
@@
 		)
 		(property "Description" ""
-			(at 486.41 61.595 0)
+			(at 486.41 31.115 0)
 			(effects
 				(font
@@
 	(symbol
 		(lib_id "power:VBUS")
-		(at 417.83 60.96 0)
+		(at 417.83 31.115 0)
 		(unit 1)
 		(exclude_from_sim no)
@@
 		(dnp no)
 		(property "Reference" "#PWR076"
-			(at 417.83 64.77 0)
+			(at 417.83 34.925 0)
 			(effects
 				(font
@@
 		)
 		(property "Value" "VBUS"
-			(at 417.83 56.515 0)
+			(at 417.83 26.67 0)
 			(effects
 				(font
@@
 		)
 		(property "Footprint" ""
-			(at 417.83 60.96 0)
+			(at 417.83 31.115 0)
 			(effects
 				(font
@@
 		)
 		(property "Datasheet" ""
-			(at 417.83 60.96 0)
+			(at 417.83 31.115 0)
 			(effects
 				(font
@@
 		)
 		(property "Description" ""
-			(at 417.83 60.96 0)
+			(at 417.83 31.115 0)
 			(effects
 				(font

Commit message: update
Connections:
- net S0: now reaches U9.10 (S0)
- net S1: now reaches U9.11 (S1)
- net S3: now reaches U9.13 (S3)
- net S2: now reaches U9.14 (S2)
- net nE: now reaches U9.15 (~{E})
Changed lines of the file:
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@@
 	(wire
 		(pts
-			(xy 420.37 292.1) (xy 430.53 292.1)
+			(xy 416.56 292.1) (xy 430.53 292.1)
 		)
 		(stroke
@@
 	(wire
 		(pts
+			(xy 430.53 302.26) (xy 416.56 302.26)
+		)
+		(stroke
+			(width 0)
+			(type default)
+		)
+	)
+	(wire
+		(pts
 			(xy 338.455 99.695) (xy 334.645 99.695)
 		)
@@
 	(wire
 		(pts
+			(xy 416.56 309.88) (xy 430.53 309.88)
+		)
+		(stroke
+			(width 0)
+			(type default)
+		)
+	)
+	(wire
+		(pts
 			(xy 269.24 203.835) (xy 283.21 203.835)
 		)
@@
 	(wire
 		(pts
+			(xy 416.56 307.34) (xy 430.53 307.34)
+		)
+		(stroke
+			(width 0)
+			(type default)
+		)
+	)
+	(wire
+		(pts
 			(xy 302.26 77.47) (xy 323.85 77.47)
 		)
@@
 	(wire
 		(pts
+			(xy 430.53 304.8) (xy 416.56 304.8)
+		)
+		(stroke
+			(width 0)
+			(type default)
+		)
+	)
+	(wire
+		(pts
 			(xy 514.985 66.675) (xy 502.285 66.675)
 		)
@@
 	(wire
 		(pts
+			(xy 416.56 320.04) (xy 430.53 320.04)
+		)
+		(stroke
+			(width 0)
+			(type default)
+		)
+	)
+	(wire
+		(pts
 			(xy 29.845 212.09) (xy 29.845 214.63)
 		)
@@
 		)
 	)
+	(label "nE"
+		(at 416.56 320.04 0)
+		(effects
+			(font
+				(size 1.27 1.27)
+			)
+			(justify left bottom)
+		)
+	)
 	(label "WS2811_12"
 		(at 421.64 84.455 0)
@@
 		)
 	)
+	(label "S3"
+		(at 416.56 309.88 0)
+		(effects
+			(font
+				(size 1.27 1.27)
+			)
+			(justify left bottom)
+		)
+	)
 	(label "IN1_L"
 		(at 554.99 198.12 180)
@@
 		)
 	)
+	(label "S0"
+		(at 416.56 302.26 0)
+		(effects
+			(font
+				(size 1.27 1.27)
+			)
+			(justify left bottom)
+		)
+	)
 	(label "LEDA8"
 		(at 269.24 156.845 0)
@@
 		)
 	)
+	(label "S2"
+		(at 416.56 307.34 0)
+		(effects
+			(font
+				(size 1.27 1.27)
+			)
+			(justify left bottom)
+		)
+	)
 	(label "LED7A_OUT"
 		(at 323.85 133.35 180)
@@
 	)
 	(label "WS2811"
-		(at 420.37 292.1 0)
+		(at 416.56 292.1 0)
 		(effects
 			(font
@@
 		)
 	)
+	(label "S1"
+		(at 416.56 304.8 0)
+		(effects
+			(font
+				(size 1.27 1.27)
+			)
+			(justify left bottom)
+		)
+	)

Commit message: update
Parts:
- removed J17: Conn_01x05_Socket, Connector_PinSocket_2.54mm:PinSocket_1x05_P2.54mm_Horizontal, symbol Connector:Conn_01x05_Socket
- removed J18: Conn_01x05_Pin, Connector_PinHeader_2.54mm:PinHeader_1x05_P2.54mm_Horizontal, symbol Connector:Conn_01x05_Pin
- removed R30, R31, R33: R0603_4.7k_1%_100mW_100PPM_AC, Resistor_SMD:R_0603_1608Metric, symbol Resistors_SMD_0603:R0603_4.7k_1%_100mW_100PPM_AC
- added R72, R73, R74, R75, R76, R77, R78, R79, R80, R81, R82, R83, R84, R85, R86: R0603_4.7k_1%_100mW_100PPM_AC, Resistor_SMD:R_0603_1608Metric, symbol Resistors_SMD_0603:R0603_4.7k_1%_100mW_100PPM_AC
Connections:
- net at R42.1, U9.6 (I3): now also R75.1
- net at R52.1, U9.22 (I9): now also R81.1
- net at R49.1, U9.17 (I14): now also R86.1
- net at R46.1, U9.23 (I8): now also R80.1
- net at R44.1, U9.5 (I4): now also R76.1
- net at R48.1, U9.19 (I12): now also R84.1
- net at R43.1, U9.7 (I2): now also R74.1
- net at R53.1, U9.20 (I11): now also R83.1
- net at R40.1, U9.9 (I0): now also R72.1
- net at R51.1, U9.2 (I7): now also R79.1
- net at J1.a12 (Pin_a12): now also J1.a18 (Pin_a18), J1.a24 (Pin_a24), J1.a30 (Pin_a30), J1.c12 (Pin_c12), J1.c18 (Pin_c18), J1.c24 (Pin_c24), J1.c30 (Pin_c30)
- net at R50.1, U9.4 (I5): now also R77.1
- net at R41.1, U9.8 (I1): now also R73.1
- net at J11.a12 (Pin_a12): now also J11.a18 (Pin_a18), J11.a24 (Pin_a24), J11.a30 (Pin_a30), J11.a6 (Pin_a6), J11.c12 (Pin_c12), J11.c18 (Pin_c18), J11.c24 (Pin_c24), J11.c30 (Pin_c30), J11.c6 (Pin_c6)
- net at R45.1, U9.3 (I6): now also R78.1
- net at R54.1, U9.18 (I13): now also R85.1
- net at R47.1, U9.21 (I10): now also R82.1
Other:
- moved on the sheet: C8

Commit message: update
Parts:
- added D1, D2, D3, D4: ESDA5V3L, Package_TO_SOT_SMD:SOT-23-3, symbol Power_Protection:ESDA5V3L
- added JP9: SolderJumper_3_Open, Jumper:SolderJumper-3_P1.3mm_Open_RoundedPad1.0x1.5mm_NumberLabels, symbol Jumper:SolderJumper_3_Open
Connections:
- net +5V: now also JP9.3 (B)
- net GND: now also D1.3 (A), D2.3 (A), D3.3 (A), D4.3 (A), JP9.1 (A)
- net 4: now reaches R42.1, R75.1, U9.6 (I3)
- net 4: now also D1.1 (K)
- net 7: now reaches R45.1, R78.1, U9.3 (I6)
- net at R78.2: now also R72.2, R73.2, R74.2, R75.2, R76.2, R77.2, R79.2, R80.2, R81.2, R82.2, R83.2, R84.2, R85.2, R86.2, JP9.2 (C)
- net 12: now reaches R53.1, R83.1, U9.20 (I11)
- net 1: now reaches R40.1, R72.1, U9.9 (I0)
- net 1: now also D4.1 (K)
- net 10: now reaches R52.1, R81.1, U9.22 (I9)
- net 10: now also D2.2 (K)
- net 15: now reaches R49.1, R86.1, U9.17 (I14)
- net 9: now reaches R46.1, R80.1, U9.23 (I8)
- net 9: now also D2.1 (K)
- net 5: now reaches R44.1, R76.1, U9.5 (I4)
- net 5: now also D1.2 (K)
- net 13: now reaches R48.1, R84.1, U9.19 (I12)
- net 3: now reaches R43.1, R74.1, U9.7 (I2)
- net 3: now also D3.2 (K)
- net 8: now reaches R51.1, R79.1, U9.2 (I7)
- net 16: now reaches R55.1, U9.16 (I15)
- net 6: now reaches R50.1, R77.1, U9.4 (I5)
- net 6: now also D3.1 (K)
- net 2: now reaches R41.1, R73.1, U9.8 (I1)
- net 2: now also D4.2 (K)
- net 14: now reaches R54.1, R85.1, U9.18 (I13)
- net 11: now reaches R47.1, R82.1, U9.21 (I10)
Other:
- moved on the sheet: R40, R41, R42, R43, R44, R45, R46, R47, R48, R49, R50, R51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

Commit message: update
Parts:
- added D5, D6: ESDA5V3L, Package_TO_SOT_SMD:SOT-23-3, symbol Power_Protection:ESDA5V3L
Connections:
- net LED15A_OUT is gone; now on net GND: J1.c28 (Pin_c28), Q15.7 (D1), Q15.8 (D1)
- net LED15B_OUT is gone; now on net GND: J1.c29 (Pin_c29), Q15.5 (D2), Q15.6 (D2)
- net WS2811_15 is gone; now on net GND: J1.c27 (Pin_c27), R49.2
- net 7: now also D5.1 (K)
- net 8: now also D5.2 (K)
- net GND: now also D5.3 (A), D6.3 (A)
- net VBUS1: now reaches J1.a12 (Pin_a12), J1.a18 (Pin_a18), J1.a24 (Pin_a24), J1.a30 (Pin_a30), J1.c12 (Pin_c12), J1.c18 (Pin_c18), J1.c24 (Pin_c24), J1.c30 (Pin_c30)
Other:
- moved on the sheet: JP9, R81, R82, R83, R84, R85, R86

Commit message: update
Parts:
- removed MOD1: ~, ZD1006:ZD1006, symbol zd1006:ZD1006
Connections:
- net 11: now also D6.1 (K)
- net 15: now also D6.2 (K)
- net GND: no longer R38.1, R39.1
- net IN4_H: now also J1.a11 (Pin_a11)
- net VBUS1: now also J11.a12 (Pin_a12), J11.a18 (Pin_a18), J11.a24 (Pin_a24), J11.a30 (Pin_a30), J11.a6 (Pin_a6), J11.c12 (Pin_c12), J11.c18 (Pin_c18), J11.c24 (Pin_c24), J11.c30 (Pin_c30), J11.c6 (Pin_c6)
- net IN4_GND: now reaches J1.c11 (Pin_c11)
- net IN4_GND: now also R39.1
