File: hardware/led_stairs_controller.kicad_pcb (KiCad board)
At the start: 4 copper layers, 100 x 83.2 mm, 60 parts, among them Q1 QM6006D, Q10 QM6006D, Q11 QM6006D, Q12 QM6006D, Q13 QM6006D, Q14 QM6006D, Q15 QM6006D, Q16 QM6006D, Q17 BSS138, Q18 BSS138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

Commit message: update
Parts:
- added JP1: SolderJumper_3_Open, Jumper:SolderJumper-3_P1.3mm_Open_RoundedPad1.0x1.5mm_NumberLabels, B.Cu at (163.9, 91.6)
- added JP2: SolderJumper_3_Open, Jumper:SolderJumper-3_P1.3mm_Open_RoundedPad1.0x1.5mm_NumberLabels, B.Cu at (167.9, 91.6)
- added JP3: SolderJumper_3_Open, Jumper:SolderJumper-3_P1.3mm_Open_RoundedPad1.0x1.5mm_NumberLabels, B.Cu at (171.9, 91.6)
Connections:
- U1 pad 1: unconnected-(U1-A0-Pad1) -> /A0
- U1 pad 2: unconnected-(U1-A1-Pad2) -> /A1
- U1 pad 24: unconnected-(U1-A5-Pad24) -> GND
- U1 pad 25: unconnected-(U1-A6-Pad25) -> GND
- U1 pad 3: unconnected-(U1-A2-Pad3) -> /A2
- U1 pad 4: unconnected-(U1-A3-Pad4) -> GND
- U1 pad 5: unconnected-(U1-A4-Pad5) -> GND
- U2 pad 21: unconnected-(U2-23-Pad21) -> /nOE
Routing:
- net /A0: track 0.00 -> 13.2 mm, vias 0 -> 1
- net /A1: track 0.00 -> 10.6 mm, vias 0 -> 1
- net GND: track 30.9 -> 40.9 mm, vias 18 -> 111
- net /A2: track 0.00 -> 9.58 mm, vias 0 -> 1
- net +5V: track 28.9 -> 31.3 mm, vias 3 -> 6
- added copper zone on B.Cu, net GND
- added copper zone on F.Cu, net GND

Commit message: update
Parts:
- moved C1 0.12 mm to (176.9, 93.9)
Routing:
- net /nOE: track 0.00 -> 34.1 mm, vias 0 -> 2
- net GND: track 40.9 -> 38.7 mm
- net /A2: track 9.58 -> 10.6 mm

Commit message: UPDATE
Parts:
- removed U4: Mini360, Mini360_step-down:Mini360_step-down
- added J1: Conn_01x04_Pin, Connector_PinHeader_2.54mm:PinHeader_1x04_P2.54mm_Vertical, F.Cu at (192.8, 90.9)
- added R22: R0603_4.7k_1%_100mW_100PPM_AC, Resistor_SMD:R_0603_1608Metric, B.Cu at (133.1, 86.4)
- added R23: R0603_4.7k_1%_100mW_100PPM_AC, Resistor_SMD:R_0603_1608Metric, B.Cu at (138.6, 86.4)
- added R24: R0805_3.01k_1%_125mW_100PPM_RC, Resistor_SMD:R_0805_2012Metric, F.Cu at (129.5, 68.8)
- added R25: R0805_3.01k_1%_125mW_100PPM_RC, Resistor_SMD:R_0805_2012Metric, F.Cu at (129.6, 74.6)
- added R26: R0603_4.7k_1%_100mW_100PPM_AC, Resistor_SMD:R_0603_1608Metric, B.Cu at (141.7, 88.5)
- added R27: R0603_4.7k_1%_100mW_100PPM_AC, Resistor_SMD:R_0603_1608Metric, B.Cu at (143.3, 88.5)
- added R28: R0805_3.01k_1%_125mW_100PPM_RC, Resistor_SMD:R_0805_2012Metric, F.Cu at (147.8, 74.6)
- added R29: R0805_3.01k_1%_125mW_100PPM_RC, Resistor_SMD:R_0805_2012Metric, F.Cu at (147.8, 68.8)
- added U3: PC817, Package_DIP:DIP-4_W7.62mm, F.Cu at (132.7, 68.8)
- added U5: PC817, Package_DIP:DIP-4_W7.62mm, F.Cu at (132.7, 74.6)
- added U6: PC817, Package_DIP:DIP-4_W7.62mm, F.Cu at (150.7, 74.6)
- added U7: PC817, Package_DIP:DIP-4_W7.62mm, F.Cu at (150.7, 68.8)
- added U8: R-78E5.0-1.0, Converter_DCDC:Converter_DCDC_RECOM_R-78E-0.5_THT, F.Cu at (111.9, 74.7)
- moved R17 4.30 mm to (152.3, 84.1)
- moved U2 4.30 mm to (130.8, 93.1)
Connections:
- MOD1 pad D2: unconnected-(MOD1-PadD2) -> /IN1_H
- MOD1 pad D5: unconnected-(MOD1-PadD5) -> /IN2_H
- U2 pad 27: unconnected-(U2-19-Pad27) -> /IN4_L
- U2 pad 28: unconnected-(U2-18-Pad28) -> /IN3_L
- U2 pad 29: unconnected-(U2-5-Pad29) -> /IN2_L
- U2 pad 30: unconnected-(U2-17-Pad30) -> /IN1_L
Routing:
- net GND: track 38.7 -> 357.3 mm, vias 111 -> 28
- net VBUS: track 0.00 -> 249.6 mm
- net +5V: track 31.3 -> 120.9 mm, vias 6 -> 7
- net /IN4_L: track 0.00 -> 56.8 mm, vias 0 -> 1
- net /IN3_L: track 0.00 -> 51.8 mm, vias 0 -> 1
- net /IN1_L: track 0.00 -> 44.5 mm, vias 0 -> 1
- net +3.3V: track 7.03 -> 48.9 mm, vias 3 -> 2
- net /IN2_L: track 0.00 -> 36.6 mm, vias 0 -> 1
- net /SDA_H: track 24.2 -> 41.9 mm, vias 0 -> 1
- net /SCL_H: track 25.4 -> 42.3 mm, vias 0 -> 1
- net /IN2_H: track 0.00 -> 16.1 mm
- net /IN1_H: track 0.00 -> 15.5 mm
- net /SDA_L: track 26.7 -> 20.4 mm
- net /nOE: track 34.1 -> 30.8 mm
- net /SCL_L: track 16.5 -> 14.0 mm
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- removed copper zone on In2.Cu, net +3.3V
- removed copper zone on In2.Cu, net +5V
- removed copper zone on In1.Cu, net GND
- removed copper zone on In2.Cu, net VBUS
Other:
- copper layers 4 -> 2

Commit message: update
Parts:
- added C2: C0603_100nF_16V_X7R, Capacitor_SMD:C_0603_1608Metric, B.Cu at (119.2, 74.7)
- added F17: Polyfuse, Fuse:Fuse_1812_4532Metric, B.Cu at (111.7, 68.3)
- added J2: Conn_01x04_Pin, Connector_PinHeader_2.54mm:PinHeader_1x04_P2.54mm_Vertical, F.Cu at (140.4, 99.9)
- added J3: Conn_01x04_Pin, Connector_PinHeader_2.54mm:PinHeader_1x04_P2.54mm_Horizontal, F.Cu at (193.0, 91.0)
- added Q19: BSS138, Package_TO_SOT_SMD:SOT-23, F.Cu at (158.0, 100.8)
- added R30: R0603_4.7k_1%_100mW_100PPM_AC, Resistor_SMD:R_0603_1608Metric, F.Cu at (182.7, 93.1)
- added R31: R0603_4.7k_1%_100mW_100PPM_AC, Resistor_SMD:R_0603_1608Metric, F.Cu at (186.0, 93.2)
- added R32: R0603_4.7k_1%_100mW_100PPM_AC, Resistor_SMD:R_0603_1608Metric, F.Cu at (164.0, 98.2)
- added U4: MCP23008-xSO, Package_SO:SOIC-18W_7.5x11.6mm_P1.27mm, F.Cu at (122.7, 94.9)
- J1: value Conn_01x04_Pin -> Conn_01x04_Socket; footprint Connector_PinHeader_2.54mm:PinHeader_1x04_P2.54mm_Vertical -> Connector_PinSocket_2.54mm:PinSocket_1x04_P2.54mm_Horizontal
- moved J1 84.3 mm to (108.5, 91.0)
- moved R29 12.5 mm to (157.1, 77.1), turned to 180 degrees
- moved R28 9.88 mm to (157.1, 71.3), turned to 180 degrees
- moved U7 8.99 mm to (154.2, 77.1), turned to 180 degrees
- moved U6 4.84 mm to (154.2, 71.3), turned to 180 degrees
Connections:
- MOD1 pad C7: /LED17_OUT -> /IN4_H
- MOD1 pad C8: /LED18_OUT -> /IN3_H
- U2 pad 21: /nOE -> /OE
- U2 pad 29: /IN2_L -> unconnected-(U2-5-Pad29)
- U2 pad 32: unconnected-(U2-4-Pad32) -> /IN2_L
- U8 pad 1: VBUS -> Net-(U8-IN)
Routing:
- net GND: track 357.3 -> 278.0 mm
- net /IN4_L: track 56.8 -> 17.1 mm
- net /IN3_L: track 51.8 -> 22.6 mm
- net /IN2_L: track 36.6 -> 14.5 mm
- net /IN1_L: track 44.5 -> 22.5 mm
- net /IN4_H: track 0.00 -> 20.3 mm
- net +5V: track 120.9 -> 141.1 mm, vias 7 -> 10
- net +3.3V: track 48.9 -> 63.2 mm
- net /IN3_H: track 0.00 -> 13.7 mm
- net /nOE: track 30.8 -> 19.7 mm
- net /OE: track 0.00 -> 10.6 mm
- net Net-(U8-IN): track 0.00 -> 7.19 mm
- net /SCL_L: track 14.0 -> 19.0 mm
- net VBUS: track 249.6 -> 245.4 mm
- net /SDA_L: track 20.4 -> 23.6 mm
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
Commit message: update
Parts:
- added C3: C0603_100nF_16V_X7R, Capacitor_SMD:C_0603_1608Metric, F.Cu at (116.1, 88.2)
- J1: value Conn_01x04_Socket -> Conn_01x05_Socket
- moved R32 20.8 mm to (184.2, 93.1)
- moved R27 15.7 mm to (127.7, 86.4), turned to -90 degrees
- moved R26 15.6 mm to (126.2, 86.4), turned to -90 degrees
- moved R23 13.9 mm to (124.7, 86.4), turned to -90 degrees
- moved R22 9.87 mm to (123.2, 86.4), turned to -90 degrees
- moved Q19 1.36 mm to (158.9, 101.8), turned to 90 degrees
- moved C2 1.10 mm to (120.3, 74.7)
- moved U8 0.83 mm to (112.8, 74.7)
- moved U4 0.74 mm to (122.0, 95.0), turned to 90 degrees
- moved R30 0.20 mm to (182.5, 93.1)
Connections:
- J1 pad 2: /SDA_H -> unconnected-(J1-Pin_2-Pad2)
- J1 pad 3: /SCL_H -> /SDA_H
- J1 pad 4: GND -> /SCL_H
- R22 pad 1: +3.3V -> P-UP
- R23 pad 1: +3.3V -> P-UP
- R26 pad 1: +3.3V -> P-UP
- R27 pad 1: +3.3V -> P-UP
- U2 pad 30: /IN1_L -> /IN2_L
- U2 pad 32: /IN2_L -> /IN1_L
- U4 pad 10: unconnected-(U4-GP0-Pad10) -> /IN4_L
- U4 pad 11: unconnected-(U4-GP1-Pad11) -> /IN3_L
- U4 pad 12: unconnected-(U4-GP2-Pad12) -> /IN2_L
- U4 pad 13: unconnected-(U4-GP3-Pad13) -> /IN1_L
- U4 pad 14: unconnected-(U4-GP4-Pad14) -> /nOE
- U4 pad 3: GND -> /A2
- U4 pad 4: GND -> /A1
- U4 pad 5: GND -> /A0
Routing:
- net /SDA_H: track 43.1 -> 147.7 mm, vias 2 -> 4
- net /SCL_H: track 44.2 -> 137.3 mm, vias 2 -> 4
- net /nOE: track 19.7 -> 82.6 mm, vias 2 -> 7
- net /A2: track 10.6 -> 63.3 mm, vias 1 -> 3
- net /A1: track 10.6 -> 60.5 mm, vias 1 -> 3
- net /A0: track 13.2 -> 59.8 mm, vias 1 -> 3
- net /IN4_L: track 17.1 -> 49.4 mm, vias 1 -> 2
- net /IN3_L: track 22.6 -> 54.3 mm, vias 1 -> 2
- net /IN2_L: track 14.5 -> 45.1 mm, vias 1 -> 2
- net +5V: track 141.1 -> 171.5 mm, vias 10 -> 12
- net /IN1_L: track 22.5 -> 50.0 mm, vias 1 -> 2
- net +3.3V: track 63.2 -> 39.3 mm
- net GND: track 278.0 -> 269.0 mm
- net P-UP: track 0.00 -> 4.50 mm
- net /OE: track 10.6 -> 8.80 mm

Commit message: update
Parts:
- added R33: R0603_4.7k_1%_100mW_100PPM_AC, Resistor_SMD:R_0603_1608Metric, F.Cu at (111.8, 91.0)
- J1: footprint Connector_PinSocket_2.54mm:PinSocket_1x04_P2.54mm_Horizontal -> Connector_PinSocket_2.54mm:PinSocket_1x05_P2.54mm_Horizontal
- J3: value Conn_01x04_Pin -> Conn_01x05_Pin; footprint Connector_PinHeader_2.54mm:PinHeader_1x04_P2.54mm_Horizontal -> Connector_PinHeader_2.54mm:PinHeader_1x05_P2.54mm_Horizontal
- moved J1 4.40 mm to (104.1, 91.0)
- moved J3 4.03 mm to (197.0, 91.0)
- moved Q19 0.69 mm to (158.9, 102.5)
Connections:
- J1 pad 2: unconnected-(J1-Pin_2-Pad2) -> /SDA_H
- J1 pad 3: /SDA_H -> /SCL_H
- J1 pad 4: /SCL_H -> /INT_H
- J3 pad 4: GND -> /INT_H
Routing:
- net /INT_H: track 0.00 -> 114.5 mm, vias 0 -> 7
- net GND: track 269.0 -> 238.7 mm
- net +5V: track 171.5 -> 185.5 mm
- net /SCL_H: track 137.3 -> 145.2 mm, vias 4 -> 5
- net /SDA_H: track 147.7 -> 154.0 mm, vias 4 -> 5
- net /IN4_L: track 49.4 -> 47.6 mm
- net /IN3_L: track 54.3 -> 53.0 mm
- net VBUS: track 245.4 -> 246.6 mm
- net /OE: track 8.80 -> 7.80 mm
