File: hardware/led_stairs_controller.kicad_pcb (KiCad board)
At the start: 2 copper layers, 100 x 83.2 mm, 103 parts, among them J1 Conn_01x05_Socket, J2 Conn_01x05_Pin, J3 Conn_01x05_Pin, Q1 QM6006D, Q10 QM6006D, Q11 QM6006D, Q12 QM6006D, Q13 QM6006D, Q14 QM6006D, Q15 QM6006D, Q16 QM6006D, Q17 BSS138, Q18 BSS138, Q19 BSS138, Q2 QM6006D, Q20 BSS138, Q3 QM6006D, Q4 QM6006D, Q5 QM6006D, Q6 QM6006D, Q7 QM6006D, Q8 QM6006D, Q9 QM6006D, U1 PCA9635, U2 ESP32-DEVKITC-32UE, U3 PC817, U4 MCP23008-xSO, U5 PC817, U6 PC817, U7 PC817, U8 R-78E5.0-1.0

Commit message: update
Parts:
- removed J2: Conn_01x05_Pin, Connector_PinHeader_2.54mm:PinHeader_1x05_P2.54mm_Vertical
- removed J3: Conn_01x05_Pin, Connector_PinHeader_2.54mm:PinHeader_1x05_P2.54mm_Horizontal
- added C8: C0603_100nF_16V_X7R, Capacitor_SMD:C_0603_1608Metric, F.Cu at (1.50, 62.5)
- added C9: C0603_100nF_16V_X7R, Capacitor_SMD:C_0603_1608Metric, F.Cu at (160.5, 88.8)
- added J11: DIN41612_02x32_AC, Connector_DIN:DIN41612_C_2x32_Male_Horizontal_THT, F.Cu at (190.5, 134.0)
- added J17: Conn_01x05_Socket, Connector_PinSocket_2.54mm:PinSocket_1x05_P2.54mm_Horizontal, F.Cu at (3.20, 136.8)
- added J18: Conn_01x05_Pin, Connector_PinHeader_2.54mm:PinHeader_1x05_P2.54mm_Horizontal, F.Cu at (22.2, 129.8)
- added J19: Conn_01x05_Pin, Connector_PinHeader_2.54mm:PinHeader_1x05_P2.54mm_Vertical, F.Cu at (-12.8, 125.3)
- added R40: R0603_4.7k_1%_100mW_100PPM_AC, Resistor_SMD:R_0603_1608Metric, F.Cu at (200.1, 128.6)
- added R41: R0603_4.7k_1%_100mW_100PPM_AC, Resistor_SMD:R_0603_1608Metric, F.Cu at (198.6, 128.6)
- added R42: R0603_4.7k_1%_100mW_100PPM_AC, Resistor_SMD:R_0603_1608Metric, F.Cu at (193.2, 118.0)
- added R43: R0603_4.7k_1%_100mW_100PPM_AC, Resistor_SMD:R_0603_1608Metric, F.Cu at (197.1, 128.6)
- added R44: R0603_4.7k_1%_100mW_100PPM_AC, Resistor_SMD:R_0603_1608Metric, F.Cu at (190.2, 118.0)
- added R45: R0603_4.7k_1%_100mW_100PPM_AC, Resistor_SMD:R_0603_1608Metric, F.Cu at (194.1, 128.6)
- added R46: R0603_4.7k_1%_100mW_100PPM_AC, Resistor_SMD:R_0603_1608Metric, F.Cu at (194.7, 118.0)
- added R47: R0603_4.7k_1%_100mW_100PPM_AC, Resistor_SMD:R_0603_1608Metric, F.Cu at (213.2, 109.8)
- added R48: R0603_4.7k_1%_100mW_100PPM_AC, Resistor_SMD:R_0603_1608Metric, F.Cu at (213.2, 112.3)
- added R49: R0603_4.7k_1%_100mW_100PPM_AC, Resistor_SMD:R_0603_1608Metric, F.Cu at (213.2, 114.8)
- added R50: R0603_4.7k_1%_100mW_100PPM_AC, Resistor_SMD:R_0603_1608Metric, F.Cu at (192.6, 128.6)
- added R51: R0603_4.7k_1%_100mW_100PPM_AC, Resistor_SMD:R_0603_1608Metric, F.Cu at (195.6, 128.6)
- added R52: R0603_4.7k_1%_100mW_100PPM_AC, Resistor_SMD:R_0603_1608Metric, F.Cu at (191.7, 118.0)
- added R53: R0603_4.7k_1%_100mW_100PPM_AC, Resistor_SMD:R_0603_1608Metric, F.Cu at (213.2, 124.9)
- added R54: R0603_4.7k_1%_100mW_100PPM_AC, Resistor_SMD:R_0603_1608Metric, F.Cu at (213.2, 127.4)
- added R55: R0603_4.7k_1%_100mW_100PPM_AC, Resistor_SMD:R_0603_1608Metric, F.Cu at (213.2, 129.9)
- added R56: R0603_1k_1%_100mW_100PPM_AC, Resistor_SMD:R_0603_1608Metric, F.Cu at (175.3, 113.1)
- added R57: R0603_1k_1%_100mW_100PPM_AC, Resistor_SMD:R_0603_1608Metric, F.Cu at (160.1, 112.9)
- added R58: R0603_1k_1%_100mW_100PPM_AC, Resistor_SMD:R_0603_1608Metric, F.Cu at (144.8, 113.0)
- added R59: R0603_1k_1%_100mW_100PPM_AC, Resistor_SMD:R_0603_1608Metric, F.Cu at (129.6, 112.9)
- added R60: R0603_1k_1%_100mW_100PPM_AC, Resistor_SMD:R_0603_1608Metric, F.Cu at (114.4, 112.9)
- added R61: R0603_1k_1%_100mW_100PPM_AC, Resistor_SMD:R_0603_1608Metric, F.Cu at (181.0, 113.1)
- added R62: R0603_1k_1%_100mW_100PPM_AC, Resistor_SMD:R_0603_1608Metric, F.Cu at (165.8, 113.0)
- added R63: R0603_1k_1%_100mW_100PPM_AC, Resistor_SMD:R_0603_1608Metric, F.Cu at (150.6, 113.0)
- added R64: R0603_1k_1%_100mW_100PPM_AC, Resistor_SMD:R_0603_1608Metric, F.Cu at (135.3, 112.9)
- added R65: R0603_1k_1%_100mW_100PPM_AC, Resistor_SMD:R_0603_1608Metric, F.Cu at (120.0, 112.9)
- added R66: R0603_1k_1%_100mW_100PPM_AC, Resistor_SMD:R_0603_1608Metric, F.Cu at (25.6, 52.4)
- added R67: R0603_1k_1%_100mW_100PPM_AC, Resistor_SMD:R_0603_1608Metric, F.Cu at (25.6, 54.9)
- added R68: R0603_1k_1%_100mW_100PPM_AC, Resistor_SMD:R_0603_1608Metric, F.Cu at (25.6, 57.5)
- added R69: R0603_1k_1%_100mW_100PPM_AC, Resistor_SMD:R_0603_1608Metric, F.Cu at (25.6, 60.0)
- added R70: R0603_1k_1%_100mW_100PPM_AC, Resistor_SMD:R_0603_1608Metric, F.Cu at (25.6, 62.5)
- added R71: R0603_1k_1%_100mW_100PPM_AC, Resistor_SMD:R_0603_1608Metric, F.Cu at (25.6, 65.0)
- added U10: PCA9635, Package_SO:TSSOP-28_4.4x9.7mm_P0.65mm, F.Cu at (161.5, 97.1)
- added U9: CD74HC4067M, Package_SO:SOIC-24W_7.5x15.4mm_P1.27mm, F.Cu at (187.3, 97.0)
- C2, C4, C5, C6, C7, F17, JP5, JP6, JP7, JP8, R1, R2, R22, R23, R26, R27, R3, R4, R5, R6, R7: moved to F.Cu
- F1, F10, F11, F12, F13, F14, F15, F16, F2, F3, F4, F5, F6, F7, F8, F9: moved to B.Cu
- J1: value Conn_01x05_Socket -> DIN41612_02x32_AC; footprint Connector_PinSocket_2.54mm:PinSocket_1x05_P2.54mm_Horizontal -> Connector_DIN:DIN41612_C_2x32_Male_Horizontal_THT
- Q1, Q10, Q11, Q12, Q13, Q14, Q15, Q16, Q2, Q3, Q4, Q5, Q6, Q7, Q8, Q9: value QM6006D -> IRF7341PBF; footprint Package_TO_SOT_SMD:TO-252-2 -> Package_SO:SOIC-8_3.9x4.9mm_P1.27mm
- moved MOD1 215.6 mm to (-111.0, 59.5)
- moved U7 203.1 mm to (-37.2, 145.0), turned to 0 degrees
- moved U6 202.8 mm to (-37.2, 138.4), turned to 0 degrees
- moved C1 180.8 mm to (1.50, 49.9)
- moved U5 179.2 mm to (-37.2, 131.7)
- moved U3 179.0 mm to (-37.2, 125.1)
- moved R32 176.0 mm to (13.5, 49.9), turned to 0 degrees
- moved R31 159.5 mm to (29.9, 126.2), turned to 0 degrees
- moved C4 156.7 mm to (1.50, 57.5)
- moved R18 155.6 mm to (9.53, 52.4), turned to 0 degrees
- moved R30 155.6 mm to (29.9, 123.7), turned to 0 degrees
- moved R21 152.6 mm to (9.53, 60.0), turned to 0 degrees
- moved R19 147.8 mm to (9.53, 54.9), turned to 0 degrees
- moved R17 146.8 mm to (9.53, 49.9)
- moved R20 146.3 mm to (9.53, 57.5), turned to 0 degrees
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Connections:
- net /LED1 renamed /LEDA1
- net /LED10 renamed /LEDA10
- net /LED11 renamed /LEDA11
- net /LED12 renamed /LEDA12
- net /LED13 renamed /LEDA13
- net /LED14 renamed /LEDA14
- net /LED15 renamed /LEDA15
- net /LED16 renamed /LEDA16
- net /LED2 renamed /LEDA2
- net /LED3 renamed /LEDA3
- net /LED4 renamed /LEDA4
- net /LED5 renamed /LEDA5
- net /LED6 renamed /LEDA6
- net /LED7 renamed /LEDA7
- net /LED8 renamed /LEDA8
- net /LED9 renamed /LEDA9
- F1 pad 1: Net-(Q1-D) -> VBUS
- F1 pad 2: /LED1_OUT -> Net-(J11-Pin_a2)
- F10 pad 1: Net-(Q10-D) -> VBUS
- F10 pad 2: /LED10_OUT -> Net-(J11-Pin_c26)
- F11 pad 1: Net-(Q11-D) -> VBUS
- F11 pad 2: /LED11_OUT -> Net-(J1-Pin_a26)
- F12 pad 1: Net-(Q12-D) -> VBUS
- F12 pad 2: /LED12_OUT -> Net-(J1-Pin_a20)
- F13 pad 1: Net-(Q13-D) -> VBUS
- F13 pad 2: /LED13_OUT -> Net-(J1-Pin_a14)
- F14 pad 1: Net-(Q14-D) -> VBUS
- F14 pad 2: /LED14_OUT -> Net-(J1-Pin_c20)
- F15 pad 1: Net-(Q15-D) -> VBUS
- F15 pad 2: /LED15_OUT -> Net-(J1-Pin_c26)
- F16 pad 1: Net-(Q16-D) -> VBUS
- F16 pad 2: /LED16_OUT -> Net-(J1-Pin_c14)
- F2 pad 1: Net-(Q2-D) -> VBUS
- F2 pad 2: /LED2_OUT -> Net-(J11-Pin_a8)
- F3 pad 1: Net-(Q3-D) -> VBUS
- F3 pad 2: /LED3_OUT -> Net-(J11-Pin_a14)
- F4 pad 1: Net-(Q4-D) -> VBUS
- F4 pad 2: /LED4_OUT -> Net-(J11-Pin_a20)
- F5 pad 1: Net-(Q5-D) -> VBUS
- F5 pad 2: /LED5_OUT -> Net-(J11-Pin_a26)
- F6 pad 1: Net-(Q6-D) -> VBUS
- F6 pad 2: /LED6_OUT -> Net-(J11-Pin_c2)
- F7 pad 1: Net-(Q7-D) -> VBUS
- F7 pad 2: /LED7_OUT -> Net-(J11-Pin_c8)
- F8 pad 1: Net-(Q8-D) -> VBUS
- F8 pad 2: /LED8_OUT -> Net-(J11-Pin_c14)
- F9 pad 1: Net-(Q9-D) -> VBUS
- F9 pad 2: /LED9_OUT -> Net-(J11-Pin_c20)
- Q1 pad 1: Net-(Q1-G) -> GND
- Q1 pad 2: Net-(Q1-D) -> Net-(Q1A-G1)
- Q10 pad 1: Net-(Q10-G) -> GND
- Q10 pad 2: Net-(Q10-D) -> Net-(Q10A-G1)
- Q11 pad 1: Net-(Q11-G) -> GND
- Q11 pad 2: Net-(Q11-D) -> Net-(Q11A-G1)
- Q12 pad 1: Net-(Q12-G) -> GND
- Q12 pad 2: Net-(Q12-D) -> Net-(Q12A-G1)
- Q13 pad 1: Net-(Q13-G) -> GND
- Q13 pad 2: Net-(Q13-D) -> Net-(Q13A-G1)
- Q14 pad 1: Net-(Q14-G) -> GND
- Q14 pad 2: Net-(Q14-D) -> Net-(Q14A-G1)
- Q15 pad 1: Net-(Q15-G) -> GND
- Q15 pad 2: Net-(Q15-D) -> Net-(Q15A-G1)
- Q16 pad 1: Net-(Q16-G) -> GND
- Q16 pad 2: Net-(Q16-D) -> Net-(Q16A-G1)
- Q2 pad 1: Net-(Q2-G) -> GND
- Q2 pad 2: Net-(Q2-D) -> Net-(Q2A-G1)
- Q3 pad 1: Net-(Q3-G) -> GND
- Q3 pad 2: Net-(Q3-D) -> Net-(Q3A-G1)
- Q4 pad 1: Net-(Q4-G) -> GND
- Q4 pad 2: Net-(Q4-D) -> Net-(Q4A-G1)
- Q5 pad 1: Net-(Q5-G) -> GND
- Q5 pad 2: Net-(Q5-D) -> Net-(Q5A-G1)
- Q6 pad 1: Net-(Q6-G) -> GND
- Q6 pad 2: Net-(Q6-D) -> Net-(Q6A-G1)
- Q7 pad 1: Net-(Q7-G) -> GND
- Q7 pad 2: Net-(Q7-D) -> Net-(Q7A-G1)
- Q8 pad 1: Net-(Q8-G) -> GND
- Q8 pad 2: Net-(Q8-D) -> Net-(Q8A-G1)
- Q9 pad 1: Net-(Q9-G) -> GND
- Q9 pad 2: Net-(Q9-D) -> Net-(Q9A-G1)
- R1 pad 2: Net-(Q1-G) -> Net-(Q1A-G1)
- R10 pad 2: Net-(Q10-G) -> Net-(Q10A-G1)
- R11 pad 2: Net-(Q11-G) -> Net-(Q11A-G1)
- R12 pad 2: Net-(Q12-G) -> Net-(Q12A-G1)
- R13 pad 2: Net-(Q13-G) -> Net-(Q13A-G1)
- R14 pad 2: Net-(Q14-G) -> Net-(Q14A-G1)
- R15 pad 2: Net-(Q15-G) -> Net-(Q15A-G1)
- R16 pad 2: Net-(Q16-G) -> Net-(Q16A-G1)
- R2 pad 2: Net-(Q2-G) -> Net-(Q2A-G1)
- R3 pad 2: Net-(Q3-G) -> Net-(Q3A-G1)
- R4 pad 2: Net-(Q4-G) -> Net-(Q4A-G1)
- R5 pad 2: Net-(Q5-G) -> Net-(Q5A-G1)
- R6 pad 2: Net-(Q6-G) -> Net-(Q6A-G1)
- R7 pad 2: Net-(Q7-G) -> Net-(Q7A-G1)
- R8 pad 2: Net-(Q8-G) -> Net-(Q8A-G1)
- R9 pad 2: Net-(Q9-G) -> Net-(Q9A-G1)
Routing:
- net +5V: track 191.0 -> 0.00 mm, vias 14 -> 0
- net /SDA_H: track 152.5 -> 0.00 mm, vias 5 -> 0
- net /SCL_H: track 144.5 -> 0.00 mm, vias 5 -> 0
- net /INT_H: track 139.0 -> 0.00 mm, vias 10 -> 0
- net GND: track 245.5 -> 148.5 mm, vias 49 -> 20
- net /nOE: track 82.3 -> 0.00 mm, vias 7 -> 0
- net /WS2811_5: track 0.00 -> 75.7 mm
- net /WS2811_10: track 0.00 -> 68.3 mm
- net /LEDA10: track 6.02 -> 72.8 mm, vias 0 -> 2
- net /LEDB10: track 0.00 -> 65.3 mm, vias 0 -> 2
- net /LEDA1: track 80.7 -> 19.5 mm, vias 1 -> 2
- net /LEDB5: track 0.00 -> 61.1 mm, vias 0 -> 2
- net Net-(U9-I0): track 0.00 -> 59.2 mm
- net /WS2811_4: track 0.00 -> 58.6 mm
- net Net-(U9-I1): track 0.00 -> 57.2 mm
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- removed copper zone on B.Cu, net GND
- removed copper zone on F.Cu, net GND
Other:
- board text removed: "${Revision}"
- board text removed: "1"
- board text removed: "JKBI"

Commit message: update
Parts:
- moved Q16 92.4 mm to (160.9, 76.0), turned to 90 degrees
- moved Q13 88.3 mm to (166.4, 76.0)
- moved F13 82.6 mm to (142.8, 57.8), turned to 0 degrees
- moved F16 81.9 mm to (144.8, 70.0), turned to 90 degrees
- moved Q14 77.4 mm to (171.9, 76.0), turned to 90 degrees
- moved Q15 72.3 mm to (183.1, 76.0), turned to 90 degrees
- moved F14 67.4 mm to (159.9, 70.1), turned to 90 degrees
- moved Q12 52.3 mm to (177.5, 76.0), turned to 90 degrees
- moved Q11 51.8 mm to (188.7, 76.0), turned to 90 degrees
- moved F15 51.6 mm to (175.2, 70.0), turned to 90 degrees
Connections:
- J1 pad a17: /LED3B_OUT -> /LED13B_OUT
- Q12 pad 5: /LED12A_OUT -> /LED12B_OUT
- Q12 pad 6: /LED12A_OUT -> /LED12B_OUT
Routing:
- net VBUS: track 190.6 -> 346.4 mm
- net /LED13A_OUT: track 0.00 -> 23.3 mm
- net /LED13B_OUT: track 0.00 -> 23.0 mm
- net /LED12B_OUT: track 0.00 -> 18.5 mm
- net /LED12A_OUT: track 0.00 -> 18.4 mm
- net /LED16B_OUT: track 0.00 -> 15.0 mm
- net /LED16A_OUT: track 0.00 -> 13.6 mm
- net /LED14B_OUT: track 0.00 -> 10.5 mm
- net /LED14A_OUT: track 0.00 -> 10.2 mm
- net Net-(U9-I7): track 47.7 -> 40.6 mm
- net Net-(J1-Pin_a14): track 0.00 -> 3.15 mm
- net Net-(J1-Pin_a26): track 0.00 -> 3.05 mm
- net Net-(J1-Pin_a20): track 0.00 -> 3.00 mm
- net Net-(J1-Pin_c20): track 0.00 -> 2.07 mm
- net Net-(J1-Pin_c14): track 0.00 -> 2.00 mm
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
Commit message: update
Parts:
- moved C1 171.1 mm to (167.4, 91.7), turned to 90 degrees
- moved R66 167.6 mm to (190.6, 81.8), turned to 90 degrees
- moved R70 160.6 mm to (184.9, 81.8), turned to 90 degrees
- moved R67 156.2 mm to (179.4, 81.8), turned to 90 degrees
- moved R69 149.9 mm to (173.8, 81.8), turned to 90 degrees
- moved R68 144.8 mm to (168.2, 81.8), turned to 90 degrees
- moved R71 138.2 mm to (162.8, 81.8), turned to 90 degrees
- moved R13 103.0 mm to (165.8, 81.8)
- moved R14 99.9 mm to (171.3, 81.8)
- moved R12 89.4 mm to (176.8, 81.8)
- moved R16 77.8 mm to (160.2, 81.8)
- moved U4 76.6 mm to (148.8, 94.6), turned to 90 degrees
- moved R11 75.7 mm to (188.1, 81.8)
- moved JP4 63.1 mm to (81.8, 90.0)
- moved R15 60.3 mm to (182.5, 81.8), turned to 90 degrees
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Connections:
- J1 pad a2: unconnected-(J1-Pin_a2-Pada2) -> VBUS
- J1 pad a7: unconnected-(J1-Pin_a7-Pada7) -> GND
- J1 pad c2: unconnected-(J1-Pin_c2-Padc2) -> VBUS
- J1 pad c7: unconnected-(J1-Pin_c7-Padc7) -> GND
Routing:
- net /WS2811_13: track 0.00 -> 45.8 mm
- net /WS2811_16: track 0.00 -> 45.8 mm
- net +5V: track 0.00 -> 39.3 mm, vias 0 -> 3
- net /WS2811_14: track 0.00 -> 30.8 mm
- net /WS2811_12: track 0.00 -> 30.4 mm
- net Net-(U9-I4): track 0.00 -> 25.6 mm, vias 0 -> 2
- net Net-(U9-I8): track 0.00 -> 23.4 mm, vias 0 -> 2
- net Net-(U9-I9): track 0.00 -> 22.3 mm, vias 0 -> 2
- net Net-(U9-I3): track 0.00 -> 20.8 mm
- net Net-(U9-I0): track 59.2 -> 39.0 mm
- net Net-(U9-I1): track 57.2 -> 37.6 mm
- net Net-(U9-I2): track 54.8 -> 36.2 mm
- net /LED11A_OUT: track 0.00 -> 16.6 mm
- net /LED11B_OUT: track 0.00 -> 16.6 mm
- net /WS2811_15: track 0.00 -> 15.4 mm
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
Commit message: update
Parts:
- moved U8 45.0 mm to (109.4, 118.4), turned to 90 degrees
Routing:
- net /LEDB11: track 0.00 -> 37.7 mm, vias 0 -> 2
- net VBUS: track 346.4 -> 381.2 mm, vias 6 -> 9
- net /LEDB15: track 0.00 -> 34.7 mm, vias 0 -> 2
- net GND: track 148.5 -> 177.9 mm, vias 20 -> 62
- net /LEDB12: track 0.00 -> 27.1 mm, vias 0 -> 2
- net /LEDA11: track 0.00 -> 24.5 mm, vias 0 -> 2
- net /LEDA15: track 0.00 -> 22.9 mm, vias 0 -> 2
- net /LEDB14: track 0.00 -> 22.9 mm, vias 0 -> 2
- net /LEDA16: track 0.00 -> 22.3 mm, vias 0 -> 2
- net /LEDA13: track 0.00 -> 19.0 mm, vias 0 -> 2
- net /LEDB13: track 0.00 -> 16.6 mm, vias 0 -> 2
- net /nOE: track 0.00 -> 14.9 mm, vias 0 -> 2
- net /LEDA12: track 0.00 -> 13.8 mm
- net /LEDB16: track 0.00 -> 12.7 mm
- net /LEDA14: track 0.00 -> 12.1 mm
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- added copper zone on B.Cu, net GND
- added copper zone on F.Cu, net GND

Commit message: update
Parts:
- moved R47 19.6 mm to (198.1, 75.1), turned to 90 degrees
- moved R48 19.1 mm to (194.9, 75.1), turned to 90 degrees
- moved R49 15.3 mm to (192.7, 69.5), turned to 90 degrees
- moved R54 13.0 mm to (194.2, 69.6), turned to 90 degrees
- moved R55 12.9 mm to (195.8, 69.6), turned to 90 degrees
- moved R53 10.1 mm to (196.5, 75.0), turned to 90 degrees
Connections:
- U9 pad 10: unconnected-(U9-S0-Pad10) -> /S0
- U9 pad 11: unconnected-(U9-S1-Pad11) -> /S1
- U9 pad 13: unconnected-(U9-S3-Pad13) -> /S3
- U9 pad 14: unconnected-(U9-S2-Pad14) -> /S2
- U9 pad 15: unconnected-(U9-~{E}-Pad15) -> /nE
Routing:
- net /S0: track 0.00 -> 41.5 mm, vias 0 -> 1
- net /S1: track 0.00 -> 35.6 mm, vias 0 -> 1
- net /S2: track 0.00 -> 32.7 mm, vias 0 -> 1
- net /nE: track 0.00 -> 32.7 mm, vias 0 -> 1
- net /S3: track 0.00 -> 31.4 mm, vias 0 -> 1
- net Net-(U9-I13): track 0.00 -> 30.6 mm
- net Net-(U9-I10): track 0.00 -> 30.2 mm
- net GND: track 177.9 -> 207.5 mm
- net Net-(U9-I15): track 0.00 -> 29.5 mm, vias 0 -> 2
- net Net-(U9-I11): track 0.00 -> 28.8 mm
- net Net-(U9-I14): track 0.00 -> 28.6 mm
- net Net-(U9-I12): track 0.00 -> 27.2 mm
- net /WS2811_11: track 15.2 -> 31.3 mm, vias 0 -> 1
- net /WS2811_12: track 30.4 -> 46.0 mm, vias 0 -> 1
- net /WS2811_13: track 45.8 -> 60.8 mm, vias 0 -> 1
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
Commit message: update
Parts:
- removed J17: Conn_01x05_Socket, Connector_PinSocket_2.54mm:PinSocket_1x05_P2.54mm_Horizontal
- removed J18: Conn_01x05_Pin, Connector_PinHeader_2.54mm:PinHeader_1x05_P2.54mm_Horizontal
- removed R30, R31, R33: R0603_4.7k_1%_100mW_100PPM_AC, Resistor_SMD:R_0603_1608Metric
- added R72: R0603_4.7k_1%_100mW_100PPM_AC, Resistor_SMD:R_0603_1608Metric, F.Cu at (195.0, 113.2)
- added R73: R0603_4.7k_1%_100mW_100PPM_AC, Resistor_SMD:R_0603_1608Metric, F.Cu at (195.0, 114.7)
- added R74: R0603_4.7k_1%_100mW_100PPM_AC, Resistor_SMD:R_0603_1608Metric, F.Cu at (194.9, 117.7)
- added R75: R0603_4.7k_1%_100mW_100PPM_AC, Resistor_SMD:R_0603_1608Metric, F.Cu at (188.0, 116.0)
- added R76: R0603_4.7k_1%_100mW_100PPM_AC, Resistor_SMD:R_0603_1608Metric, F.Cu at (188.0, 117.5)
- added R77: R0603_4.7k_1%_100mW_100PPM_AC, Resistor_SMD:R_0603_1608Metric, F.Cu at (194.9, 116.2)
- added R78: R0603_4.7k_1%_100mW_100PPM_AC, Resistor_SMD:R_0603_1608Metric, F.Cu at (202.9, 113.8)
- added R79: R0603_4.7k_1%_100mW_100PPM_AC, Resistor_SMD:R_0603_1608Metric, F.Cu at (204.9, 117.9)
- added R80: R0603_4.7k_1%_100mW_100PPM_AC, Resistor_SMD:R_0603_1608Metric, F.Cu at (188.0, 113.0)
- added R81: R0603_4.7k_1%_100mW_100PPM_AC, Resistor_SMD:R_0603_1608Metric, F.Cu at (188.0, 114.5)
- added R82: R0603_4.7k_1%_100mW_100PPM_AC, Resistor_SMD:R_0603_1608Metric, F.Cu at (210.8, 117.2)
- added R83: R0603_4.7k_1%_100mW_100PPM_AC, Resistor_SMD:R_0603_1608Metric, F.Cu at (210.8, 119.7)
- added R84: R0603_4.7k_1%_100mW_100PPM_AC, Resistor_SMD:R_0603_1608Metric, F.Cu at (214.8, 107.2)
- added R85: R0603_4.7k_1%_100mW_100PPM_AC, Resistor_SMD:R_0603_1608Metric, F.Cu at (214.8, 109.7)
- added R86: R0603_4.7k_1%_100mW_100PPM_AC, Resistor_SMD:R_0603_1608Metric, F.Cu at (214.8, 112.2)
- C2, C6, C7, F17, JP5, JP6, JP7, JP8: moved to B.Cu
- moved U7 192.6 mm to (139.9, 69.4), turned to -90 degrees
- moved C8 188.9 mm to (185.2, 106.3), turned to 90 degrees
- moved U3 179.4 mm to (133.3, 69.5), turned to -90 degrees
- moved U5 175.3 mm to (126.7, 69.5), turned to -90 degrees
- moved U6 171.7 mm to (120.0, 69.5), turned to -90 degrees
- moved C5 162.4 mm to (157.4, 105.4)
- moved R39 161.6 mm to (156.2, 42.2), turned to 90 degrees
- moved R38 157.4 mm to (153.3, 42.2), turned to 90 degrees
- moved R37 153.3 mm to (150.3, 42.2), turned to 90 degrees
- moved R36 149.1 mm to (147.4, 42.2), turned to 90 degrees
- moved R29 144.9 mm to (144.4, 42.2), turned to 90 degrees
- moved R28 140.8 mm to (141.5, 42.2), turned to 90 degrees
- moved R25 136.6 mm to (138.6, 42.2), turned to 90 degrees
- moved R24 132.4 mm to (135.6, 42.2), turned to 90 degrees
- moved C2 126.3 mm to (112.2, 113.3), turned to 180 degrees
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Connections:
- J1 pad a12: unconnected-(J1-Pin_a12-Pada12) -> Net-(J1-Pin_a12)
- J1 pad a18: unconnected-(J1-Pin_a18-Pada18) -> Net-(J1-Pin_a12)
- J1 pad a24: unconnected-(J1-Pin_a24-Pada24) -> Net-(J1-Pin_a12)
- J1 pad a30: unconnected-(J1-Pin_a30-Pada30) -> Net-(J1-Pin_a12)
- J1 pad c12: unconnected-(J1-Pin_c12-Padc12) -> Net-(J1-Pin_a12)
- J1 pad c18: unconnected-(J1-Pin_c18-Padc18) -> Net-(J1-Pin_a12)
- J1 pad c24: unconnected-(J1-Pin_c24-Padc24) -> Net-(J1-Pin_a12)
- J1 pad c30: unconnected-(J1-Pin_c30-Padc30) -> Net-(J1-Pin_a12)
- J11 pad a12: unconnected-(J11-Pin_a12-Pada12) -> Net-(J11-Pin_a12)
- J11 pad a18: unconnected-(J11-Pin_a18-Pada18) -> Net-(J11-Pin_a12)
- J11 pad a24: unconnected-(J11-Pin_a24-Pada24) -> Net-(J11-Pin_a12)
- J11 pad a30: unconnected-(J11-Pin_a30-Pada30) -> Net-(J11-Pin_a12)
- J11 pad a6: unconnected-(J11-Pin_a6-Pada6) -> Net-(J11-Pin_a12)
- J11 pad c12: unconnected-(J11-Pin_c12-Padc12) -> Net-(J11-Pin_a12)
- J11 pad c18: unconnected-(J11-Pin_c18-Padc18) -> Net-(J11-Pin_a12)
- J11 pad c24: unconnected-(J11-Pin_c24-Padc24) -> Net-(J11-Pin_a12)
- J11 pad c30: unconnected-(J11-Pin_c30-Padc30) -> Net-(J11-Pin_a12)
- J11 pad c6: unconnected-(J11-Pin_c6-Padc6) -> Net-(J11-Pin_a12)
Routing:
- net Net-(J11-Pin_a12): track 0.00 -> 107.0 mm
- net +5V: track 46.3 -> 119.4 mm
- net Net-(J1-Pin_a12): track 0.00 -> 70.5 mm
- net /A2: track 14.8 -> 46.0 mm
- net /A1: track 13.9 -> 41.7 mm
- net /A0: track 12.8 -> 38.8 mm
- net Net-(U9-I3): track 20.9 -> 28.3 mm, vias 0 -> 2
- net VBUS: track 381.2 -> 388.5 mm
- net Net-(U8-IN): track 0.00 -> 6.05 mm
- net GND: track 207.5 -> 212.6 mm, vias 62 -> 112
- net Net-(U9-I8): track 23.4 -> 27.7 mm, vias 2 -> 4
- net Net-(U9-I9): track 22.3 -> 26.4 mm, vias 2 -> 4
- net Net-(U9-I4): track 25.6 -> 29.7 mm
- net /WS2811_4: track 69.6 -> 66.9 mm
- net /WS2811_10: track 77.0 -> 74.3 mm
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Other:
- board text added: "JP1 A0 JP2 A1 JP3 A2"

Commit message: update
Parts:
- added D1: ESDA5V3L, Package_TO_SOT_SMD:SOT-23-3, B.Cu at (187.6, 116.8)
- added D2: ESDA5V3L, Package_TO_SOT_SMD:SOT-23-3, B.Cu at (187.6, 113.4)
- added D3: ESDA5V3L, Package_TO_SOT_SMD:SOT-23-3, B.Cu at (194.5, 117.0)
- added D4: ESDA5V3L, Package_TO_SOT_SMD:SOT-23-3, B.Cu at (194.4, 113.5)
- added JP9: SolderJumper_3_Open, Jumper:SolderJumper-3_P1.3mm_Open_RoundedPad1.0x1.5mm_NumberLabels, B.Cu at (186.7, 109.3)
- moved C3 145.9 mm to (143.8, 87.0), turned to -90 degrees
- moved R17 86.1 mm to (89.8, 81.0)
- moved R18 86.1 mm to (89.8, 83.6)
- moved R20 86.1 mm to (89.8, 88.6)
- moved R21 86.1 mm to (89.8, 91.1)
- moved R23 86.1 mm to (89.8, 96.1)
- moved R26 86.1 mm to (89.8, 98.6)
- moved R27 86.1 mm to (89.8, 101.1)
- moved R32 86.1 mm to (93.8, 81.0)
- moved R34 86.1 mm to (93.8, 86.1)
- moved R35 86.1 mm to (93.8, 88.6)
- moved R19 86.1 mm to (89.8, 86.1)
- moved R22 86.1 mm to (89.8, 93.6)
- moved R82 42.0 mm to (204.6, 75.6)
- moved R83 42.0 mm to (204.6, 78.1)
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Connections:
- net Net-(U9-I0) renamed /1
- net Net-(U9-I1) renamed /2
- net Net-(U9-I10) renamed /11
- net Net-(U9-I11) renamed /12
- net Net-(U9-I12) renamed /13
- net Net-(U9-I13) renamed /14
- net Net-(U9-I14) renamed /15
- net Net-(U9-I15) renamed /16
- net Net-(U9-I2) renamed /3
- net Net-(U9-I3) renamed /4
- net Net-(U9-I4) renamed /5
- net Net-(U9-I5) renamed /6
- net Net-(U9-I6) renamed /7
- net Net-(U9-I7) renamed /8
- net Net-(U9-I8) renamed /9
- net Net-(U9-I9) renamed /10
- R72 pad 2: unconnected-(R72-Pad2) -> Net-(JP9-C)
- R73 pad 2: unconnected-(R73-Pad2) -> Net-(JP9-C)
- R74 pad 2: unconnected-(R74-Pad2) -> Net-(JP9-C)
- R75 pad 2: unconnected-(R75-Pad2) -> Net-(JP9-C)
- R76 pad 2: unconnected-(R76-Pad2) -> Net-(JP9-C)
- R77 pad 2: unconnected-(R77-Pad2) -> Net-(JP9-C)
- R78 pad 2: unconnected-(R78-Pad2) -> Net-(JP9-C)
- R79 pad 2: unconnected-(R79-Pad2) -> Net-(JP9-C)
- R80 pad 2: unconnected-(R80-Pad2) -> Net-(JP9-C)
- R81 pad 2: unconnected-(R81-Pad2) -> Net-(JP9-C)
- R82 pad 2: unconnected-(R82-Pad2) -> Net-(JP9-C)
- R83 pad 2: unconnected-(R83-Pad2) -> Net-(JP9-C)
- R84 pad 2: unconnected-(R84-Pad2) -> Net-(JP9-C)
- R85 pad 2: unconnected-(R85-Pad2) -> Net-(JP9-C)
- R86 pad 2: unconnected-(R86-Pad2) -> Net-(JP9-C)
Routing:
- net Net-(J11-Pin_a12): track 107.0 -> 165.8 mm
- net Net-(JP9-C): track 0.00 -> 23.6 mm, vias 0 -> 3
- net unconnected-(J11-Pin_a1-Pada1): track 0.00 -> 18.7 mm
- net GND: track 212.6 -> 229.6 mm, vias 112 -> 201
- net unconnected-(J11-Pin_c1-Padc1): track 0.00 -> 14.2 mm
- net +3.3V: track 2.23 -> 11.8 mm
- net +5V: track 119.4 -> 126.2 mm
- net /1: track 39.0 -> 44.1 mm, vias 0 -> 2
- net /2: track 37.6 -> 42.2 mm, vias 0 -> 2
- net /3: track 36.2 -> 40.1 mm, vias 0 -> 2
- net /6: track 32.0 -> 34.2 mm, vias 2 -> 3
- net /4: track 28.3 -> 29.6 mm
- net /5: track 29.7 -> 30.6 mm, vias 2 -> 3
- net /9: track 27.7 -> 28.4 mm

Commit message: update
Parts:
- added D5: ESDA5V3L, Package_TO_SOT_SMD:SOT-23-3, B.Cu at (194.4, 109.9)
- added D6: ESDA5V3L, Package_TO_SOT_SMD:SOT-23-3, B.Cu at (198.4, 85.3)
- R25: moved to B.Cu
- moved U3 53.0 mm to (89.2, 40.2), turned to 0 degrees
- moved R24 49.9 mm to (92.3, 67.1)
- moved R25 40.4 mm to (107.3, 67.8)
- moved R39 31.0 mm to (144.4, 70.9), turned to -90 degrees
- moved R29 28.7 mm to (146.3, 70.9), turned to -90 degrees
- moved U6 16.0 mm to (135.2, 74.5), turned to 0 degrees
- moved R82 12.4 mm to (198.0, 86.1)
- moved R84 11.8 mm to (198.0, 80.1)
- moved R86 11.6 mm to (198.0, 84.5)
- moved R85 11.3 mm to (198.1, 81.6)
- moved U7 10.2 mm to (148.7, 74.6), turned to 0 degrees
- moved R83 8.24 mm to (198.0, 83.0)
- moved U5 0.60 mm to (126.6, 70.1)
- moved R78 0.38 mm to (195.0, 109.1)
- moved R79 0.38 mm to (195.0, 110.7)
Routing:
- net /WS2811: track 0.00 -> 55.1 mm, vias 0 -> 1
- net Net-(JP9-C): track 23.6 -> 64.2 mm
- net unconnected-(J11-Pin_a1-Pada1): track 18.7 -> 0.00 mm
- net unconnected-(J11-Pin_c1-Padc1): track 14.2 -> 0.56 mm
- net /IN4_L: track 0.00 -> 12.3 mm
- net /IN3_L: track 0.00 -> 9.34 mm
- net GND: track 229.6 -> 236.9 mm, vias 201 -> 206
- net Net-(R39-Pad2): track 0.00 -> 7.09 mm
- net /S1: track 35.6 -> 40.5 mm
- net Net-(R29-Pad2): track 0.00 -> 4.40 mm
- net /8: track 29.6 -> 33.0 mm, vias 0 -> 2
- net /7: track 31.0 -> 33.8 mm, vias 2 -> 4
- net VBUS: track 388.5 -> 385.7 mm
- net +5V: track 126.2 -> 124.0 mm
- net /LEDB1: track 26.5 -> 25.0 mm
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Other:
- board size 100 x 83.2 mm -> 100 x 83.7 mm
