File: hardware/led_stairs_controller.kicad_pcb (KiCad board)
At the start: 2 copper layers, 100 x 83.7 mm, 158 parts, among them J1 DIN41612_02x32_AC, J11 DIN41612_02x32_AC, J19 Conn_01x05_Pin, Q1 IRF7341PBF, Q10 IRF7341PBF, Q11 IRF7341PBF, Q12 IRF7341PBF, Q13 IRF7341PBF, Q14 IRF7341PBF, Q15 IRF7341PBF, Q16 IRF7341PBF, Q17 BSS138, Q18 BSS138, Q19 BSS138, Q2 IRF7341PBF, Q20 BSS138, Q3 IRF7341PBF, Q4 IRF7341PBF, Q5 IRF7341PBF, Q6 IRF7341PBF, Q7 IRF7341PBF, Q8 IRF7341PBF, Q9 IRF7341PBF, U1 PCA9635, U10 PCA9635, U2 ESP32-DEVKITC-32UE, U3 PC817, U4 MCP23008-xSO, U5 PC817, U6 PC817, U7 PC817, U8 R-78E5.0-1.0, U9 CD74HC4067M

Commit message: update
Parts:
- removed MOD1: ~, ZD1006:ZD1006
- moved U6 0.76 mm to (136.0, 74.5)
Connections:
- D6 pad 1: unconnected-(D6-K-Pad1) -> /11
- D6 pad 2: unconnected-(D6-K-Pad2) -> /15
- J1 pad a11: unconnected-(J1-Pin_a11-Pada11) -> /IN4_H
- J1 pad a12: Net-(J1-Pin_a12) -> VBUS1
- J1 pad a18: Net-(J1-Pin_a12) -> VBUS1
- J1 pad a24: Net-(J1-Pin_a12) -> VBUS1
- J1 pad a30: Net-(J1-Pin_a12) -> VBUS1
- J1 pad c11: unconnected-(J1-Pin_c11-Padc11) -> /IN4_GND
- J1 pad c12: Net-(J1-Pin_a12) -> VBUS1
- J1 pad c18: Net-(J1-Pin_a12) -> VBUS1
- J1 pad c24: Net-(J1-Pin_a12) -> VBUS1
- J1 pad c27: /WS2811_15 -> GND
- J1 pad c28: /LED15A_OUT -> GND
- J1 pad c29: /LED15B_OUT -> GND
- J1 pad c30: Net-(J1-Pin_a12) -> VBUS1
- J11 pad a12: Net-(J11-Pin_a12) -> VBUS1
- J11 pad a18: Net-(J11-Pin_a12) -> VBUS1
- J11 pad a24: Net-(J11-Pin_a12) -> VBUS1
- J11 pad a30: Net-(J11-Pin_a12) -> VBUS1
- J11 pad a6: Net-(J11-Pin_a12) -> VBUS1
- J11 pad c12: Net-(J11-Pin_a12) -> VBUS1
- J11 pad c18: Net-(J11-Pin_a12) -> VBUS1
- J11 pad c24: Net-(J11-Pin_a12) -> VBUS1
- J11 pad c30: Net-(J11-Pin_a12) -> VBUS1
- J11 pad c6: Net-(J11-Pin_a12) -> VBUS1
- Q15 pad 5: /LED15B_OUT -> GND
- Q15 pad 6: /LED15B_OUT -> GND
- Q15 pad 7: /LED15A_OUT -> GND
- Q15 pad 8: /LED15A_OUT -> GND
- R38 pad 1: GND -> unconnected-(R38-Pad1)
- R39 pad 1: GND -> /IN4_GND
- R49 pad 2: /WS2811_15 -> GND
Routing:
- net VBUS1: track 0.00 -> 279.6 mm
- net Net-(J11-Pin_a12): track 165.4 -> 0.00 mm
- net Net-(J1-Pin_a12): track 70.5 -> 0.00 mm
- net GND: track 236.9 -> 274.6 mm, vias 206 -> 207
- net /WS2811_15: track 19.3 -> 0.00 mm, vias 1 -> 0
- net /SCL_H: track 12.7 -> 30.8 mm, vias 2 -> 3
- net /nOE: track 14.9 -> 32.8 mm, vias 2 -> 3
- net /IN4_H: track 0.00 -> 16.4 mm
- net /SDA_H: track 13.8 -> 29.5 mm, vias 2 -> 3
- net /IN4_GND: track 0.00 -> 9.96 mm
- net /LED15A_OUT: track 9.23 -> 0.00 mm
- net /LED15B_OUT: track 9.23 -> 0.00 mm
- net +5V: track 124.0 -> 130.7 mm, vias 4 -> 5
- net /15: track 28.6 -> 34.7 mm, vias 0 -> 2
- net /10: track 26.4 -> 29.2 mm
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
Commit message: update
Parts:
- R25: moved to F.Cu
- moved U3 42.1 mm to (113.7, 74.4)
- moved R26 40.8 mm to (129.1, 88.0), turned to 90 degrees
- moved R38 34.1 mm to (134.7, 70.8), turned to -90 degrees
- moved R36 32.7 mm to (131.6, 70.8), turned to -90 degrees
- moved R17 30.6 mm to (111.2, 102.8), turned to 90 degrees
- moved R28 29.1 mm to (136.7, 70.9), turned to -90 degrees
- moved Q17 26.1 mm to (114.3, 91.6), turned to -90 degrees
- moved R25 22.7 mm to (129.7, 70.8), turned to -90 degrees
- moved JP4 18.2 mm to (112.5, 102.6), turned to 0 degrees
- moved Q18 14.1 mm to (122.3, 91.3), turned to -90 degrees
- moved Q19 13.7 mm to (118.4, 91.4), turned to -90 degrees
- moved U5 4.71 mm to (124.8, 74.5), turned to 0 degrees
- moved Q20 3.81 mm to (126.3, 91.5), turned to -90 degrees
- moved R29 2.30 mm to (148.7, 70.9)
- moved R39 2.00 mm to (146.4, 70.8)
Connections:
- J1 pad a10: unconnected-(J1-Pin_a10-Pada10) -> /IN3_H
- J1 pad a8: unconnected-(J1-Pin_a8-Pada8) -> /IN1_H
- J1 pad a9: unconnected-(J1-Pin_a9-Pada9) -> /IN2_H
- J1 pad c10: unconnected-(J1-Pin_c10-Padc10) -> /IN3_GND
- J1 pad c8: unconnected-(J1-Pin_c8-Padc8) -> /IN1_GND
- J1 pad c9: unconnected-(J1-Pin_c9-Padc9) -> /IN2_GND
- R38 pad 1: unconnected-(R38-Pad1) -> /IN3_GND
Routing:
- net /IN3_L: track 9.02 -> 22.1 mm
- net /IN3_H: track 0.00 -> 10.0 mm
- net Net-(R38-Pad2): track 0.00 -> 6.49 mm
- net /IN3_GND: track 0.00 -> 4.04 mm
- net /14: track 30.6 -> 34.6 mm, vias 0 -> 2
- net Net-(R28-Pad2): track 0.00 -> 3.04 mm
- net /13: track 27.2 -> 29.4 mm, vias 0 -> 2
- net /IN4_H: track 16.4 -> 18.2 mm
- net /IN4_GND: track 9.96 -> 11.7 mm
- net /12: track 28.9 -> 30.6 mm, vias 0 -> 2
- net Net-(R29-Pad2): track 4.40 -> 2.83 mm
- net Net-(R39-Pad2): track 7.09 -> 6.36 mm

Commit message: update
Parts:
- removed U4: MCP23008-xSO, Package_SO:SOIC-18W_7.5x11.6mm_P1.27mm
- added D7: ESDA5V3L, Package_TO_SOT_SMD:SOT-23-3, B.Cu at (198.4, 81.9)
- added JP12: SolderJumper_3_Open, Jumper:SolderJumper-3_P1.3mm_Open_RoundedPad1.0x1.5mm_NumberLabels, F.Cu at (144.2, 70.0)
- added JP13: Jumper_2_Open, Jumper:SolderJumper-2_P1.3mm_Open_RoundedPad1.0x1.5mm, F.Cu at (141.2, 71.3)
- added JP14: Jumper_2_Open, Jumper:SolderJumper-2_P1.3mm_Open_RoundedPad1.0x1.5mm, F.Cu at (141.3, 68.7)
- added R30: R0603_4.7k_1%_100mW_100PPM_AC, Resistor_SMD:R_0603_1608Metric, F.Cu at (206.9, 75.1)
- added U11: MCP23017_SO, Package_SO:SOIC-28W_7.5x17.9mm_P1.27mm, F.Cu at (145.7, 94.7)
- moved R22 46.2 mm to (135.7, 88.4), turned to 90 degrees
- moved R23 45.1 mm to (134.2, 88.4), turned to 90 degrees
- moved R18 39.3 mm to (125.4, 100.0), turned to -90 degrees
- moved R37 39.1 mm to (124.2, 71.3), turned to 180 degrees
- moved R27 38.9 mm to (126.5, 88.5), turned to 90 degrees
- moved R21 38.4 mm to (126.8, 101.1), turned to -90 degrees
- moved R32 36.4 mm to (126.9, 96.2), turned to 90 degrees
- moved R35 32.8 mm to (125.5, 97.0), turned to 90 degrees
- moved R24 32.0 mm to (124.2, 69.3), turned to 180 degrees
- moved R20 16.8 mm to (105.7, 93.7)
- moved R19 16.7 mm to (105.7, 91.2)
- moved R34 12.2 mm to (105.7, 88.7)
- moved Q18 11.4 mm to (117.8, 101.8), turned to 0 degrees
- moved Q20 9.14 mm to (117.8, 94.8), turned to 0 degrees
- moved Q17 7.52 mm to (117.8, 98.3), turned to 0 degrees
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Connections:
- J1 pad a10: /IN3_H -> GND
- J1 pad a11: /IN4_H -> /IN4
- J1 pad a12: VBUS1 -> VBUS
- J1 pad a8: /IN1_H -> VBUS
- J1 pad a9: /IN2_H -> /IN3_H
- J1 pad c10: /IN3_GND -> unconnected-(J1-Pin_c10-Padc10)
- J1 pad c11: /IN4_GND -> unconnected-(J1-Pin_c11-Padc11)
- J1 pad c12: VBUS1 -> unconnected-(J1-Pin_c12-Padc12)
- J1 pad c8: /IN1_GND -> unconnected-(J1-Pin_c8-Padc8)
- J1 pad c9: /IN2_GND -> unconnected-(J1-Pin_c9-Padc9)
Routing:
- net /IN1_L: track 0.00 -> 68.9 mm, vias 0 -> 1
- net /IN2_L: track 0.00 -> 61.6 mm, vias 0 -> 5
- net /IN4_L: track 11.7 -> 51.5 mm, vias 0 -> 3
- net /SDA_L: track 0.00 -> 38.2 mm
- net /IN3_L: track 22.1 -> 58.4 mm, vias 0 -> 3
- net /SDA_H: track 29.5 -> 62.3 mm, vias 3 -> 5
- net /SCL_L: track 0.00 -> 31.9 mm
- net /SCL_H: track 30.8 -> 62.4 mm, vias 3 -> 5
- net +3.3V: track 11.8 -> 38.4 mm, vias 0 -> 3
- net /nOE: track 32.8 -> 59.4 mm, vias 3 -> 4
- net +5V: track 130.7 -> 155.2 mm, vias 5 -> 7
- net /INT_L: track 0.00 -> 15.4 mm
- net /IN4: track 0.00 -> 14.4 mm
- net /OE: track 0.00 -> 14.3 mm
- net Net-(R37-Pad2): track 0.00 -> 14.1 mm
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
Commit message: update
Parts:
- removed JP12: SolderJumper_3_Open, Jumper:SolderJumper-3_P1.3mm_Open_RoundedPad1.0x1.5mm_NumberLabels
- removed JP13, JP14: Jumper_2_Open, Jumper:SolderJumper-2_P1.3mm_Open_RoundedPad1.0x1.5mm
- added D8: ESDA5V3L, Package_TO_SOT_SMD:SOT-23-3, B.Cu at (198.4, 78.5)
- added J2: Conn_01x05_Pin, jumper:Jumper 5, B.Cu at (138.5, 63.3)
- added J3: Conn_01x05_Pin, jumper:Jumper 5, B.Cu at (138.4, 68.0)
- added J4: Conn_01x05_Pin, jumper:Jumper 5, B.Cu at (126.7, 63.8)
- added J5: Conn_01x05_Pin, jumper:Jumper 5, B.Cu at (126.7, 67.6)
- moved R30 9.30 mm to (198.0, 77.7)
- moved R28 1.83 mm to (138.6, 70.8)
- moved R39 1.62 mm to (146.3, 73.8)
- moved C4 1.28 mm to (107.9, 102.8), turned to 180 degrees
- moved R38 1.08 mm to (135.8, 70.7)
- moved R47 0.75 mm to (198.1, 74.3)
- moved R48 0.73 mm to (195.0, 74.4)
- moved R53 0.65 mm to (196.5, 74.3)
- moved R84 0.48 mm to (198.0, 79.2)
- moved JP4 0.38 mm to (112.5, 102.2)
Connections:
- J1 pad a9: /IN3_H -> unconnected-(J1-Pin_a9-Pada9)
- J1 pad c10: unconnected-(J1-Pin_c10-Padc10) -> GND
- J1 pad c11: unconnected-(J1-Pin_c11-Padc11) -> /IN3
- J1 pad c12: unconnected-(J1-Pin_c12-Padc12) -> VBUS
- J1 pad c27: GND -> /WS2811_15
- J1 pad c28: GND -> /LED15A_OUT
- J1 pad c29: GND -> /LED15B_OUT
- J1 pad c8: unconnected-(J1-Pin_c8-Padc8) -> VBUS
- Q15 pad 5: GND -> /LED15B_OUT
- Q15 pad 6: GND -> /LED15B_OUT
- Q15 pad 7: GND -> /LED15A_OUT
- Q15 pad 8: GND -> /LED15A_OUT
- R36 pad 1: GND -> /IN2_GND
- R37 pad 1: GND -> /IN1_GND
- R49 pad 2: GND -> /WS2811_15
Routing:
- net +5V: track 155.2 -> 191.2 mm, vias 7 -> 8
- net P-UP: track 0.00 -> 34.8 mm, vias 0 -> 1
- net GND: track 271.9 -> 239.9 mm, vias 210 -> 250
- net /WS2811: track 55.1 -> 80.8 mm
- net /INT_H: track 7.31 -> 30.3 mm
- net /nOE: track 59.4 -> 76.2 mm, vias 4 -> 3
- net /WS2811_15: track 0.00 -> 16.6 mm, vias 0 -> 1
- net /IN4_GND: track 4.46 -> 19.4 mm, vias 0 -> 1
- net /S1: track 40.5 -> 55.2 mm, vias 1 -> 2
- net /S0: track 41.1 -> 55.3 mm, vias 1 -> 2
- net /S3: track 31.3 -> 43.7 mm, vias 1 -> 2
- net /IN4: track 14.4 -> 2.46 mm
- net /S2: track 32.2 -> 43.8 mm, vias 1 -> 2
- net /IN1_H: track 10.5 -> 0.00 mm
- net VBUS: track 385.7 -> 396.2 mm
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Other:
- board text added: "10 5"
- board text added: "11 15"
- board text added: "12 14"
- board text added: "13 16"
- board text added: "6 1"
- board text added: "7 2"
- board text added: "8 3"
- board text added: "9 4"
- board text added: "A"
- board text added: "B"
- board text added: "D"
- board text added: "GND"
- board text added: "VBUS"
- board text added: "VBUS1"

Commit message: update
Parts:
- moved J4 6.59 mm to (133.3, 63.3)
- moved J5 6.50 mm to (133.2, 68.2)
- moved R21 6.30 mm to (120.5, 101.1)
- moved R32 6.10 mm to (121.7, 93.0)
- moved R35 5.25 mm to (120.4, 95.6)
- moved R18 4.46 mm to (121.7, 97.5)
- moved R28 3.41 mm to (135.2, 71.4), turned to 180 degrees
- moved R36 2.78 mm to (128.9, 71.4), turned to 180 degrees
- moved J3 2.08 mm to (140.5, 68.2)
- moved J2 2.08 mm to (140.6, 63.2)
- moved R25 1.67 mm to (128.9, 69.4), turned to 180 degrees
- moved R38 1.45 mm to (135.2, 69.4), turned to 180 degrees
Connections:
- J1 pad a10: GND -> VBUS
- J1 pad a11: /IN4 -> GND
- J1 pad a12: VBUS -> /IN4
- J1 pad a13: GND -> VBUS
- J1 pad a6: unconnected-(J1-Pin_a6-Pada6) -> VBUS1
- J1 pad a8: VBUS -> GND
- J1 pad a9: unconnected-(J1-Pin_a9-Pada9) -> /IN2
- J1 pad c10: GND -> VBUS
- J1 pad c11: /IN3 -> GND
- J1 pad c12: VBUS -> /IN3
- J1 pad c13: GND -> VBUS
- J1 pad c6: unconnected-(J1-Pin_c6-Padc6) -> VBUS1
- J1 pad c8: VBUS -> GND
- J1 pad c9: unconnected-(J1-Pin_c9-Padc9) -> /IN1
Routing:
- net +5V: track 191.2 -> 176.2 mm, vias 8 -> 7
- net /IN4_GND: track 19.4 -> 8.96 mm, vias 1 -> 0
- net GND: track 239.9 -> 234.8 mm, vias 250 -> 248
- net /SCL_H: track 63.8 -> 60.1 mm
- net /IN4_H: track 17.8 -> 14.5 mm, vias 1 -> 0
- net /SDA_H: track 64.0 -> 60.7 mm
- net /IN4: track 2.46 -> 0.00 mm
- net /IN3: track 2.14 -> 0.18 mm
- net VBUS: track 396.2 -> 394.3 mm
- net /IN3_H: track 1.86 -> 0.00 mm, vias 1 -> 0
- net /IN3_GND: track 1.77 -> 0.00 mm, vias 1 -> 0
- net +3.3V: track 40.0 -> 39.4 mm
- net P-UP: track 34.8 -> 34.2 mm

Commit message: update
Parts:
- moved R22 1.60 mm to (134.1, 88.4)
- moved R23 1.52 mm to (135.7, 88.4)
Connections:
- R22 pad 2: /IN1_L -> /IN2_L
- R23 pad 2: /IN2_L -> /IN1_L
- R24 pad 1: /IN1_H -> /IN2_H
- R25 pad 1: /IN2_H -> /IN1_H
- R36 pad 1: /IN2_GND -> /IN1_GND
- R37 pad 1: /IN1_GND -> /IN2_GND
- U3 pad 4: /IN1_L -> /IN2_L
- U5 pad 4: /IN2_L -> /IN1_L
Routing:
- net /IN2_GND: track 0.00 -> 13.9 mm, vias 0 -> 1
- net +5V: track 176.2 -> 189.8 mm, vias 7 -> 10
- net VBUS: track 394.3 -> 407.8 mm
- net GND: track 234.8 -> 248.3 mm, vias 248 -> 315
- net /IN2_H: track 0.00 -> 13.1 mm, vias 0 -> 3
- net /IN2_L: track 63.1 -> 73.9 mm
- net /IN1_L: track 69.3 -> 58.5 mm
- net /IN4_GND: track 8.96 -> 17.3 mm, vias 0 -> 1
- net VBUS1: track 272.9 -> 281.1 mm
- net /IN3_H: track 0.00 -> 6.59 mm, vias 0 -> 1
- net /IN3_GND: track 0.00 -> 4.55 mm, vias 0 -> 1
- net /IN1_H: track 0.00 -> 4.44 mm, vias 0 -> 1
- net /IN1_GND: track 0.00 -> 3.53 mm, vias 0 -> 1
- net Net-(R38-Pad2): track 6.45 -> 9.77 mm
- net /IN4: track 0.00 -> 2.70 mm
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