File: hardware/_autosave-led_stairs_controller.kicad_sch (KiCad schematic)
At the start: 164 parts, among them J1 DIN41612_02x32_AC, J11 DIN41612_02x32_AC, J19 Conn_01x05_Pin, J2 Conn_01x05_Pin, J3 Conn_01x05_Pin, J4 Conn_01x05_Pin, J5 Conn_01x05_Pin, Q1 IRF7341PBF, Q10 IRF7341PBF, Q11 IRF7341PBF, Q12 IRF7341PBF, Q13 IRF7341PBF, Q14 IRF7341PBF, Q15 IRF7341PBF, Q16 IRF7341PBF, Q17 BSS138, Q18 BSS138, Q19 BSS138, Q2 IRF7341PBF, Q20 BSS138, Q3 IRF7341PBF, Q4 IRF7341PBF, Q5 IRF7341PBF, Q6 IRF7341PBF, Q7 IRF7341PBF, Q8 IRF7341PBF, Q9 IRF7341PBF, U1 PCA9635, U10 PCA9635, U11 MCP23017_SO, U2 ESP32-DEVKITC-32UE, U3 PC817, U5 PC817, U6 PC817, U7 PC817, U8 R-78E5.0-1.0, U9 CD74HC4067M

Commit message: update
Connections:
- net IN1: now also J1.c9 (Pin_c9)
- net IN1_H: no longer J1.c9 (Pin_c9)
- net IN2: now also J1.a9 (Pin_a9)
- net IN2_H: no longer J1.a9 (Pin_a9)
- net VBUS1: now also J1.a6 (Pin_a6), J1.c6 (Pin_c6)
Changed lines of the file:
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@@
 	)
 	(junction
+		(at 463.55 46.355)
+		(diameter 0)
+		(color 0 0 0 0)
+	)
+	(junction
 		(at 417.83 56.515)
 		(diameter 0)
@@
 	)
 	(junction
+		(at 440.69 46.355)
+		(diameter 0)
+		(color 0 0 0 0)
+	)
+	(junction
 		(at 417.83 64.135)
 		(diameter 0)
@@
 	(wire
 		(pts
+			(xy 440.69 46.355) (xy 440.69 76.835)
+		)
+		(stroke
+			(width 0)
+			(type default)
+		)
+	)
+	(wire
+		(pts
 			(xy 313.055 202.565) (xy 327.025 202.565)
 		)
@@
 	(wire
 		(pts
-			(xy 440.69 31.75) (xy 440.69 76.835)
+			(xy 440.69 31.75) (xy 440.69 46.355)
 		)
 		(stroke
@@
 	(wire
 		(pts
-			(xy 463.55 31.75) (xy 463.55 76.835)
+			(xy 463.55 31.75) (xy 463.55 46.355)
 		)
 		(stroke
@@
 	(wire
 		(pts
+			(xy 463.55 46.355) (xy 463.55 76.835)
+		)
+		(stroke
+			(width 0)
+			(type default)
+		)
+	)
+	(wire
+		(pts
 			(xy 546.1 200.66) (xy 560.07 200.66)
 		)
@@
 	(wire
 		(pts
+			(xy 440.69 46.355) (xy 445.77 46.355)
+		)
+		(stroke
+			(width 0)
+			(type default)
+		)
+	)
+	(wire
+		(pts
 			(xy 542.925 36.195) (xy 550.545 36.195)
 		)
@@
 	(wire
 		(pts
+			(xy 458.47 46.355) (xy 463.55 46.355)
+		)
+		(stroke
+			(width 0)
+			(type default)
+		)
+	)
+	(wire
+		(pts
 			(xy 433.705 270.51) (xy 433.705 276.225)
 		)
@@
 		)
 	)
-	(label "IN1_H"
+	(label "IN1"
 		(at 483.87 53.975 180)
 		(effects
@@
 		)
 	)
-	(label "IN2_H"
+	(label "IN2"
 		(at 420.37 53.975 0)
 		(effects
